Commit message: Changed the models within the visual mesh folder. Then updated the macro.xacro and the urdf files with the corresponding new .stl files. Also cleaned the urdf folder a little by deliting base_link (which is an unnecessary file in this package).

File: fanuc_config/urdf/m10iA.urdf (robot description, URDF)
Before this commit: robot m10iA, 8 links, 7 joints
Links:
- link base_link: geometry collision mesh filename=package://fanuc_config/meshes/m_10iA/collision/base_link.stl; visual mesh filename=package://fanuc_config/meshes/m_10iA/visual/base_link.stl
- link link_1: geometry collision mesh filename=package://fanuc_config/meshes/m_10iA/collision/link_1.stl; visual mesh filename=package://fanuc_config/meshes/m_10iA/visual/link_1.stl
- link link_2: geometry collision mesh filename=package://fanuc_config/meshes/m_10iA/collision/link_2.stl; visual mesh filename=package://fanuc_config/meshes/m_10iA/visual/link_2.stl
- link link_3: geometry collision mesh filename=package://fanuc_config/meshes/m_10iA/collision/link_3.stl; visual mesh filename=package://fanuc_config/meshes/m_10iA/visual/link_3.stl
- link link_4: geometry collision mesh filename=package://fanuc_config/meshes/m_10iA/collision/link_4.stl; visual mesh filename=package://fanuc_config/meshes/m_10iA/visual/link_4.stl
- link link_5: geometry collision mesh filename=package://fanuc_config/meshes/m_10iA/collision/link_5.stl; visual mesh filename=package://fanuc_config/meshes/m_10iA/visual/link_5.stl
- link link_6: geometry collision mesh filename=package://fanuc_config/meshes/m_10iA/collision/link_6.stl; visual mesh filename=package://fanuc_config/meshes/m_10iA/visual/link_6.stl

File: fanuc_config/urdf/m_10iA_macro.xacro (robot description, xacro)
@@ -10,5 +10,5 @@
       			<geometry>
         			<mesh
-          			filename="package://fanuc_config/meshes/m_10iA/visual/base_link.STL" />
+          			filename="package://fanuc_config/meshes/m_10iA/visual/base_link.stl" />
       			</geometry>
       			<material
@@ -37,5 +37,5 @@
       			<geometry>
         			<mesh
-          			filename="package://fanuc_config/meshes/m_10iA/visual/link_1.STL" />
+          			filename="package://fanuc_config/meshes/m_10iA/visual/link_1.stl" />
       			</geometry>
       			<material name="grey"/>
@@ -58,5 +58,5 @@
       			<geometry>
         			<mesh
-          			filename="package://fanuc_config/meshes/m_10iA/visual/link_2.STL" />
+          			filename="package://fanuc_config/meshes/m_10iA/visual/link_2.stl" />
       			</geometry>
       			<material name="grey"/>
@@ -79,5 +79,5 @@
 			  	<geometry>
 					<mesh
-				  	filename="package://fanuc_config/meshes/m_10iA/visual/link_3.STL" />
+				  	filename="package://fanuc_config/meshes/m_10iA/visual/link_3.stl" />
 			  	</geometry>
 			  	<material name="grey"/>
@@ -100,5 +100,5 @@
 				  <geometry>
 					<mesh
-					  filename="package://fanuc_config/meshes/m_10iA/visual/link_4.STL" />
+					  filename="package://fanuc_config/meshes/m_10iA/visual/link_4.stl" />
 				  </geometry>
 				  <material name="grey"/>
@@ -121,5 +121,5 @@
 				<geometry>
 					<mesh
-					  filename="package://fanuc_config/meshes/m_10iA/visual/link_5.STL" />
+					  filename="package://fanuc_config/meshes/m_10iA/visual/link_5.stl" />
 				</geometry>
 				<material name="grey"/>
@@ -142,5 +142,5 @@
 				<geometry>
 					<mesh
-					  filename="package://fanuc_config/meshes/m_10iA/visual/link_6.STL" />
+					  filename="package://fanuc_config/meshes/m_10iA/visual/link_6.stl" />
 				</geometry>
 				<material name="grey"/>
