Commit message: Added prefix to joint elements in m430iA2F macro

File: fanuc_config/urdf/m_430iA2F_macro.xacro (robot description, xacro)
@@ -109,6 +109,6 @@
         <joint name="${prefix}joint_1" type="revolute">
             <origin xyz="-6.0758E-19 1.2493E-16 0.44" rpy="0 0 0" />
-            <parent link="base_link" />
-            <child link="link_1" />
+            <parent link="${prefix}base_link" />
+            <child link="${prefix}link_1" />
             <axis xyz="0 0 1" />
             <limit lower="-3.1415" upper="3.1415" effort="0"
@@ -121,6 +121,6 @@
         <joint name="${prefix}joint_2" type="revolute">
             <origin xyz="-1.4097E-17 0.171 -4.4409E-16" rpy="0 0 0" />
-            <parent link="link_1" />
-            <child link="link_2" />
+            <parent link="${prefix}link_1" />
+            <child link="${prefix}link_2" />
             <axis xyz="0 1 0" />
             <limit lower="-2.00707" upper="2.00707" effort="0"
@@ -134,6 +134,6 @@
             <!-- origin xyz="1.2197E-19 -0.171 0.403" rpy="0 0 0" / -->
             <origin xyz="1.2197E-19 -0.171 0.350" rpy="0 0 0" />
-            <parent link="link_2" />
-            <child link="link_3" />
+            <parent link="${prefix}link_2" />
+            <child link="${prefix}link_3" />
             <axis xyz="0 1 0" />
             <limit lower="-1.771457" upper="1.771457" effort="0"
@@ -147,6 +147,6 @@
             <!-- origin xyz="-2.6075E-17 -0.06 0.497" rpy="0 0 0" / -->
             <origin xyz="-2.6075E-17 -0.06 0.55" rpy="0 0 0" />
-            <parent link="link_3" />
-            <child link="link_4" />
+            <parent link="${prefix}link_3" />
+            <child link="${prefix}link_4" />
             <axis xyz="0 1 0" />
             <limit lower="-2.617917" upper="2.617917" effort="0"
@@ -159,6 +159,6 @@
 		<joint name="${prefix}joint_5" type="revolute">
 			<origin xyz="1.4734E-16 -0.035 0.065" rpy="0 0 0" />
-			<parent link="link_4" />
-			<child link="link_5" />
+			<parent link="${prefix}link_4" />
+			<child link="${prefix}link_5" />
 			<axis xyz="0 0 1" />
 			<limit lower="-4.71225" upper="4.71225" effort="0"
@@ -170,6 +170,6 @@
 		</joint>
         <joint name="${prefix}joint_5-tool0" type="fixed">
-            <parent link="${prefix}link_5"/>
-            <child link="${prefix}tool0"/>
+            <parent link="${prefix}${prefix}link_5"/>
+            <child link="${prefix}${prefix}tool0"/>
             <origin xyz="0 0 0" rpy="0 0 0"/>
         </joint>

Commit message: Fix copy/pasta double prefix

File: fanuc_config/urdf/m_430iA2F_macro.xacro (robot description, xacro)
@@ -170,6 +170,6 @@
 		</joint>
         <joint name="${prefix}joint_5-tool0" type="fixed">
-            <parent link="${prefix}${prefix}link_5"/>
-            <child link="${prefix}${prefix}tool0"/>
+            <parent link="${prefix}link_5"/>
+            <child link="${prefix}tool0"/>
             <origin xyz="0 0 0" rpy="0 0 0"/>
         </joint>
