Commit message: Changed file name for visual models to match standard directory structure.

File: fanuc_config/urdf/M16iB20.urdf (robot description, URDF)
Before this commit: robot M16iB20, 8 links, 7 joints
Links:
- link Link_1: geometry collision mesh filename=package://fanuc_config/meshes/m_16iB20/collision/Link_1.STL; visual mesh filename=package://fanuc_config/meshes/m_16iB20/visual/Link_1.STL
- link Link_2: geometry collision mesh filename=package://fanuc_config/meshes/m_16iB20/collision/Link_2.STL; visual mesh filename=package://fanuc_config/meshes/m_16iB20/visual/Link_2.STL
- link Link_3: geometry collision mesh filename=package://fanuc_config/meshes/m_16iB20/collision/Link_3.STL; visual mesh filename=package://fanuc_config/meshes/m_16iB20/visual/Link_3.STL
- link Link_4: geometry collision mesh filename=package://fanuc_config/meshes/m_16iB20/collision/Link_4.STL; visual mesh filename=package://fanuc_config/meshes/m_16iB20/visual/Link_4.STL
- link Link_5: geometry collision mesh filename=package://fanuc_config/meshes/m_16iB20/collision/Link_5.STL; visual mesh filename=package://fanuc_config/meshes/m_16iB20/visual/Link_5.STL
- link Link_6: geometry collision mesh filename=package://fanuc_config/meshes/m_16iB20/collision/Link_6.STL; visual mesh filename=package://fanuc_config/meshes/m_16iB20/visual/Link_6.STL
- link base_link: geometry collision mesh filename=package://fanuc_config/meshes/m_16iB20/collision/base_link.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; visual mesh filename=package://fanuc_config/meshes/m_16iB20/visual/base_link.STL

File: fanuc_config/urdf/M16iB20_macro.xacro (robot description, xacro)
@@ -24,5 +24,5 @@
 		      <geometry>
 			<mesh
-			  filename="package://fanuc_config/meshes/m_16iB20/visualization/base_link.STL" />
+			  filename="package://fanuc_config/meshes/m_16iB20/visual/base_link.STL" />
 		      </geometry>
 		      <material
@@ -63,5 +63,5 @@
 		      <geometry>
 			<mesh
-			  filename="package://fanuc_config/meshes/m_16iB20/visualization/Link_1.STL" />
+			  filename="package://fanuc_config/meshes/m_16iB20/visual/Link_1.STL" />
 		      </geometry>
 		      <material
@@ -102,5 +102,5 @@
 		      <geometry>
 			<mesh
-			  filename="package://fanuc_config/meshes/m_16iB20/visualization/Link_2.STL" />
+			  filename="package://fanuc_config/meshes/m_16iB20/visual/Link_2.STL" />
 		      </geometry>
 		      <material
@@ -141,5 +141,5 @@
 		      <geometry>
 			<mesh
-			  filename="package://fanuc_config/meshes/m_16iB20/visualization/Link_3.STL" />
+			  filename="package://fanuc_config/meshes/m_16iB20/visual/Link_3.STL" />
 		      </geometry>
 		      <material
@@ -180,5 +180,5 @@
 		      <geometry>
 			<mesh
-			  filename="package://fanuc_config/meshes/m_16iB20/visualization/Link_4.STL" />
+			  filename="package://fanuc_config/meshes/m_16iB20/visual/Link_4.STL" />
 		      </geometry>
 		      <material
@@ -219,5 +219,5 @@
 		      <geometry>
 			<mesh
-			  filename="package://fanuc_config/meshes/m_16iB20/visualization/Link_5.STL" />
+			  filename="package://fanuc_config/meshes/m_16iB20/visual/Link_5.STL" />
 		      </geometry>
 		      <material
@@ -258,5 +258,5 @@
 		      <geometry>
 			<mesh
-			  filename="package://fanuc_config/meshes/m_16iB20/visualization/Link_6.STL" />
+			  filename="package://fanuc_config/meshes/m_16iB20/visual/Link_6.STL" />
 		      </geometry>
 		      <material

Commit message: Updated M16iB20 joint velocity limits based on website data (http://tr.fanucrobotics.eu/en/products/a_industrial-robots/m-16ib).  This check in addresses issue #35.

File: fanuc_config/urdf/M16iB20.urdf (robot description, URDF)
Before this commit: robot M16iB20, 8 links, 7 joints
Joints:
- joint Joint_1: limit lower=-2.967 upper=2.967 effort=0 velocity=0 -> lower=-2.967 upper=2.967 effort=0 velocity=2.8
- joint Joint_2: limit lower=-1.5708 upper=1.9 effort=0 velocity=0 -> lower=-1.5708 upper=1.9 effort=0 velocity=2.8
- joint Joint_3: limit lower=-4.21 upper=1.45 effort=0 velocity=0 -> lower=-4.21 upper=1.45 effort=0 velocity=3.0
- joint Joint_4: limit lower=-3.4907 upper=3.4907 effort=0 velocity=0 -> lower=-3.4907 upper=3.4907 effort=0 velocity=6.1
- joint Joint_5: limit lower=-2.4435 upper=2.4435 effort=0 velocity=0 -> lower=-2.4435 upper=2.4435 effort=0 velocity=5.9
- joint Joint_6: limit lower=-7.85398 upper=7.85398 effort=0 velocity=0 -> lower=-7.85398 upper=7.85398 effort=0 velocity=9.0

File: fanuc_config/urdf/M16iB20_macro.xacro (robot description, xacro)
@@ -292,5 +292,5 @@
 		      upper="2.967"
 		      effort="0"
-		      velocity="0" />
+		      velocity="2.8" />
 		    <calibration
 		      rising="0"
@@ -319,5 +319,5 @@
 		      upper="1.9"
 		      effort="0"
-		      velocity="0" />
+		      velocity="2.8" />
 		    <calibration
 		      rising="0"
@@ -346,5 +346,5 @@
 		      upper="1.45"
 		      effort="0"
-		      velocity="0" />
+		      velocity="3.0" />
 		    <calibration
 		      rising="0"
@@ -373,5 +373,5 @@
 		      upper="3.4907"
 		      effort="0"
-		      velocity="0" />
+		      velocity="6.1" />
 		    <calibration
 		      rising="0"
@@ -400,5 +400,5 @@
 		      upper="2.4435"
 		      effort="0"
-		      velocity="0" />
+		      velocity="5.9" />
 		    <calibration
 		      rising="0"
@@ -427,5 +427,5 @@
 		      upper="7.85398"
 		      effort="0"
-		      velocity="0" />
+		      velocity="9.0" />
 		    <calibration
 		      rising="0"

Commit message: Merged in changes from fuerte_dev branch revisions 1083-1111 (inclusive).  Required quite a bit of hand merging due to directory renaming.

File: fanuc_config/urdf/M16iB20.urdf (robot description, URDF)
Before this commit: robot M16iB20, 8 links, 7 joints
Links:
- removed link Link_1
- removed link Link_2
- removed link Link_3
- removed link Link_4
- removed link Link_5
- removed link Link_6
- added link link_1, mass 48654.354928172; collision mesh filename=package://fanuc_config/meshes/m_16iB20/collision/Link_1.STL; visual mesh filename=package://fanuc_config/meshes/m_16iB20/visual/Link_1.STL
- added link link_2, mass 48654.354928172; collision mesh filename=package://fanuc_config/meshes/m_16iB20/collision/Link_2.STL; visual mesh filename=package://fanuc_config/meshes/m_16iB20/visual/Link_2.STL
- added link link_3, mass 48654.354928172; collision mesh filename=package://fanuc_config/meshes/m_16iB20/collision/Link_3.STL; visual mesh filename=package://fanuc_config/meshes/m_16iB20/visual/Link_3.STL
- added link link_4, mass 48654.354928172; collision mesh filename=package://fanuc_config/meshes/m_16iB20/collision/Link_4.STL; visual mesh filename=package://fanuc_config/meshes/m_16iB20/visual/Link_4.STL
- added link link_5, mass 48654.354928172; collision mesh filename=package://fanuc_config/meshes/m_16iB20/collision/Link_5.STL; visual mesh filename=package://fanuc_config/meshes/m_16iB20/visual/Link_5.STL
- added link link_6, mass 48654.354928172; collision mesh filename=package://fanuc_config/meshes/m_16iB20/collision/Link_6.STL; visual mesh filename=package://fanuc_config/meshes/m_16iB20/visual/Link_6.STL
Joints:
- removed joint Joint_1
- removed joint Joint_2
- removed joint Joint_3
- removed joint Joint_4
- removed joint Joint_5
- removed joint Joint_6
- removed joint Joint_6-tool0
- added joint joint_1: type revolute, parent base_link, child link_1, origin xyz=0 0 0.24477 rpy=0 0 0, axis 0 0 1, limit lower=-2.967 upper=2.967 effort=0 velocity=2.8
- added joint joint_2: type revolute, parent link_1, child link_2, origin xyz=0.15 0.18759 0.28 rpy=0 0 0, axis 0 1 0, limit lower=-1.39 upper=2.78 effort=0 velocity=2.8
- added joint joint_3: type revolute, parent link_2, child link_3, origin xyz=0 -0.18815 0.77 rpy=0 0 0, axis 0 -1 0, limit lower=-4.21 upper=1.45 effort=0 velocity=3.0
- added joint joint_4: type revolute, parent link_3, child link_4, origin xyz=0.1847 0 0.1 rpy=0 0 0, axis -1 0 0, limit lower=-3.48 upper=3.48 effort=0 velocity=6.1
- added joint joint_5: type revolute, parent link_4, child link_5, origin xyz=0.55575 0.00019326 0.00073427 rpy=0 0 0, axis 0 -1 0, limit lower=-2.44 upper=2.44 effort=0 velocity=5.9
- added joint joint_6: type revolute, parent link_5, child link_6, origin xyz=0.10014 0 0.00013231 rpy=0 0 0, axis -1 0 -0.0013212, limit lower=-7.85 upper=7.85 effort=0 velocity=9.0
- added joint joint_6-tool0: type fixed, parent link_6, child tool0, origin xyz=0 0 0 rpy=0 0 0

File: fanuc_config/urdf/M16iB20_macro.xacro (robot description, xacro)
@@ -42,5 +42,5 @@
 		    </collision>
 		  </link>
-		  <link name="${prefix}Link_1">
+		  <link name="${prefix}link_1">
 		    <inertial>
 		      <origin
@@ -81,5 +81,5 @@
 		    </collision>
 		  </link>
-		  <link name="${prefix}Link_2">
+		  <link name="${prefix}link_2">
 		    <inertial>
 		      <origin
@@ -120,5 +120,5 @@
 		    </collision>
 		  </link>
-		  <link name="${prefix}Link_3">
+		  <link name="${prefix}link_3">
 		    <inertial>
 		      <origin
@@ -159,5 +159,5 @@
 		    </collision>
 		  </link>
-		  <link name="${prefix}Link_4">
+		  <link name="${prefix}link_4">
 		    <inertial>
 		      <origin
@@ -198,5 +198,5 @@
 		    </collision>
 		  </link>
-		  <link name="${prefix}Link_5">
+		  <link name="${prefix}link_5">
 		    <inertial>
 		      <origin
@@ -237,5 +237,5 @@
 		    </collision>
 		  </link>
-		  <link name="${prefix}Link_6">
+		  <link name="${prefix}link_6">
 		    <inertial>
 		      <origin
@@ -278,5 +278,5 @@
         	  <link name="${prefix}tool0"/>
 	<!-- joints -->
-		  <joint name="${prefix}Joint_1" type="revolute">
+		  <joint name="${prefix}joint_1" type="revolute">
 		    <origin
 		      xyz="0 0 0.24477"
@@ -285,5 +285,5 @@
 		      link="base_link" />
 		    <child
-		      link="Link_1" />
+		      link="link_1" />
 		    <axis
 		      xyz="0 0 1" />
@@ -305,44 +305,44 @@
 		      k_velocity="0" /-->
 		  </joint>
-		  <joint name="${prefix}Joint_2" type="revolute">
+		  <joint name="${prefix}joint_2" type="revolute">
 		    <origin
 		      xyz="0.15 0.18759 0.28"
 		      rpy="0 0 0" />
 		    <parent
-		      link="Link_1" />
-		    <child
-		      link="Link_2" />
+		      link="link_1" />
+		    <child
+		      link="link_2" />
+		    <axis
+		      xyz="0 1 0" />
+		    <limit
+		      lower="-1.38"
+		      upper="2.78"
+		      effort="0"
+		      velocity="2.8" />
+		    <calibration
+		      rising="0"
+		      falling="0" />
+		    <dynamics
+		      damping="0"
+		      friction="0" />
+		    <!--safety_controller
+		      soft_lower_limit="0"
+		      soft_upper_limit="0"
+		      k_position="0"
+		      k_velocity="0" /-->
+		  </joint>
+		  <joint name="${prefix}joint_3" type="revolute">
+		    <origin
+		      xyz="0 -0.18815 0.77"
+		      rpy="0 0 0" />
+		    <parent
+		      link="link_2" />
+		    <child
+		      link="link_3" />
 		    <axis
 		      xyz="0 -1 0" />
 		    <limit
-		      lower="-1.5708"
-		      upper="1.9"
-		      effort="0"
-		      velocity="2.8" />
-		    <calibration
-		      rising="0"
-		      falling="0" />
-		    <dynamics
-		      damping="0"
-		      friction="0" />
-		    <!--safety_controller
-		      soft_lower_limit="0"
-		      soft_upper_limit="0"
-		      k_position="0"
-		      k_velocity="0" /-->
-		  </joint>
-		  <joint name="${prefix}Joint_3" type="revolute">
-		    <origin
-		      xyz="0 -0.18815 0.77"
-		      rpy="0 0 0" />
-		    <parent
-		      link="Link_2" />
-		    <child
-		      link="Link_3" />
-		    <axis
-		      xyz="0 1 0" />
-		    <limit
-		      lower="-4.21"
-		      upper="1.45"
+		      lower="4.08"
+		      upper="1.38"
 		      effort="0"
 		      velocity="3.0" />
@@ -359,17 +359,17 @@
 		      k_velocity="0" /-->
 		  </joint>
-		  <joint name="${prefix}Joint_4" type="revolute">
+		  <joint name="${prefix}joint_4" type="revolute">
 		    <origin
 		      xyz="0.1847 0 0.1"
 		      rpy="0 0 0" />
 		    <parent
-		      link="Link_3" />
-		    <child
-		      link="Link_4" />
-		    <axis
-		      xyz="-1 0 -0.0013212" />
-		    <limit
-		      lower="-3.4907"
-		      upper="3.4907"
+		      link="link_3" />
+		    <child
+		      link="link_4" />
+		    <axis
+		      xyz="-1 0 0" />
+		    <limit
+		      lower="-3.48"
+		      upper="3.48"
 		      effort="0"
 		      velocity="6.1" />
@@ -386,17 +386,17 @@
 		      k_velocity="0" /-->
 		  </joint>
-		  <joint name="${prefix}Joint_5" type="revolute">
+		  <joint name="${prefix}joint_5" type="revolute">
 		    <origin
 		      xyz="0.55575 0.00019326 0.00073427"
 		      rpy="0 0 0" />
 		    <parent
-		      link="Link_4" />
-		    <child
-		      link="Link_5" />
-		    <axis
-		      xyz="0 1 0" />
-		    <limit
-		      lower="-2.4435"
-		      upper="2.4435"
+		      link="link_4" />
+		    <child
+		      link="link_5" />
+		    <axis
+		      xyz="0 -1 0" />
+		    <limit
+		      lower="-2.43"
+		      upper="2.43"
 		      effort="0"
 		      velocity="5.9" />
@@ -413,17 +413,17 @@
 		      k_velocity="0" /-->
 		  </joint>
-		  <joint name="${prefix}Joint_6" type="revolute">
+		  <joint name="${prefix}joint_6" type="revolute">
 		    <origin
 		      xyz="0.10014 0 0.00013231"
 		      rpy="0 0 0" />
 		    <parent
-		      link="Link_5" />
-		    <child
-		      link="Link_6" />
-		    <axis
-		      xyz="-1 0 -0.0013212" />
-		    <limit
-		      lower="-7.85398"
-		      upper="7.85398"
+		      link="link_5" />
+		    <child
+		      link="link_6" />
+		    <axis
+		      xyz="-1 0 0" />
+		    <limit
+		      lower="-7.84"
+		      upper="7.84"
 		      effort="0"
 		      velocity="9.0" />
@@ -440,6 +440,6 @@
 		      k_velocity="0" /-->
 		  </joint>
-		  <joint name="${prefix}Joint_6-tool0" type="fixed">
-		      <parent link="${prefix}Link_6"/>
+		  <joint name="${prefix}joint_6-tool0" type="fixed">
+		      <parent link="${prefix}link_6"/>
 	              <child link="${prefix}tool0"/>
           	      <origin xyz="0 0 0" rpy="0 0 0"/>

Commit message: update M16iB20 urdf (joint positions, axis directions) to match datasheet.  Regenerate meshes, arm_navigation package to match.  Add IKFast analytic IK solution.

File: fanuc_config/urdf/M16iB20.urdf (robot description, URDF)
Before this commit: robot M16iB20, 8 links, 7 joints
Links:
- link base_link: mass 48654.354928172 -> None
- link link_1: mass 48654.354928172 -> None
- link link_2: mass 48654.354928172 -> None
- link link_3: mass 48654.354928172 -> None
- link link_4: mass 48654.354928172 -> None
- link link_5: mass 48654.354928172 -> None
- link link_6: mass 48654.354928172 -> None
Joints:
- joint joint_1: limit lower=-2.967 upper=2.967 effort=0 velocity=2.8 -> lower=-2.967 upper=2.967 effort=0 velocity=2.879; origin xyz=0 0 0.24477 rpy=0 0 0 -> xyz=0 0 0.245 rpy=0 0 0
- joint joint_2: limit lower=-1.39 upper=2.78 effort=0 velocity=2.8 -> lower=-1.38 upper=2.78 effort=0 velocity=2.879
- joint joint_3: limit lower=-4.21 upper=1.45 effort=0 velocity=3.0 -> lower=-4.08 upper=1.38 effort=0 velocity=3.054; origin xyz=0 -0.18815 0.77 rpy=0 0 0 -> xyz=0 -0.18759 0.77 rpy=0 0 0
- joint joint_4: limit lower=-3.48 upper=3.48 effort=0 velocity=6.1 -> lower=-3.48 upper=3.48 effort=0 velocity=6.108; origin xyz=0.1847 0 0.1 rpy=0 0 0 -> xyz=0.18425 0 0.1 rpy=0 0 0
- joint joint_5: limit lower=-2.44 upper=2.44 effort=0 velocity=5.9 -> lower=-2.43 upper=2.43 effort=0 velocity=5.934; origin xyz=0.55575 0.00019326 0.00073427 rpy=0 0 0 -> xyz=0.55575 0 0 rpy=0 0 0
- joint joint_6: axis -1 0 -0.0013212 -> -1 0 0; limit lower=-7.85 upper=7.85 effort=0 velocity=9.0 -> lower=-7.84 upper=7.84 effort=0 velocity=9.075; origin xyz=0.10014 0 0.00013231 rpy=0 0 0 -> xyz=0.1 0 0 rpy=0 0 0

File: fanuc_config/urdf/M16iB20_macro.xacro (robot description, xacro)
@@ -4,18 +4,4 @@
 	<!-- links -->
 		  <link name="${prefix}base_link">
-		    <inertial>
-		      <origin
-			xyz="0 9.68920591007408E-05 0.538248432765216"
-			rpy="0 0 0" />
-		      <mass
-			value="48654.354928172" />
-		      <inertia
-			ixx="51563.7946245021"
-			ixy="0.552841467322453"
-			ixz="-212.267889356987"
-			iyy="49495.9076886951"
-			iyz="1.80688027777408"
-			izz="54368.3241585813" />
-		    </inertial>
 		    <visual>
 		      <origin
@@ -43,18 +29,4 @@
 		  </link>
 		  <link name="${prefix}link_1">
-		    <inertial>
-		      <origin
-			xyz="0.0335399435995477 9.68920591007463E-05 0.293476071945811"
-			rpy="0 0 0" />
-		      <mass
-			value="48654.354928172" />
-		      <inertia
-			ixx="51563.7946245021"
-			ixy="0.552841467322453"
-			ixz="-212.267889356987"
-			iyy="49495.9076886951"
-			iyz="1.80688027777408"
-			izz="54368.3241585813" />
-		    </inertial>
 		    <visual>
 		      <origin
@@ -82,18 +54,4 @@
 		  </link>
 		  <link name="${prefix}link_2">
-		    <inertial>
-		      <origin
-			xyz="-0.116459985096576 -0.187496105761522 0.0134762050463809"
-			rpy="0 0 0" />
-		      <mass
-			value="48654.354928172" />
-		      <inertia
-			ixx="51563.7946245021"
-			ixy="0.552841467322453"
-			ixz="-212.267889356987"
-			iyy="49495.9076886951"
-			iyz="1.80688027777408"
-			izz="54368.3241585813" />
-		    </inertial>
 		    <visual>
 		      <origin
@@ -121,18 +79,4 @@
 		  </link>
 		  <link name="${prefix}link_3">
-		    <inertial>
-		      <origin
-			xyz="-0.116459985097232 0.000649393837860671 -0.7565234388513"
-			rpy="0 0 0" />
-		      <mass
-			value="48654.354928172" />
-		      <inertia
-			ixx="51563.7946245021"
-			ixy="0.552841467322453"
-			ixz="-212.267889356987"
-			iyy="49495.9076886951"
-			iyz="1.80688027777408"
-			izz="54368.3241585813" />
-		    </inertial>
 		    <visual>
 		      <origin
@@ -160,18 +104,4 @@
 		  </link>
 		  <link name="${prefix}link_4">
-		    <inertial>
-		      <origin
-			xyz="-0.301157421773673 0.000649393837861561 -0.856523437562654"
-			rpy="0 0 0" />
-		      <mass
-			value="48654.354928172" />
-		      <inertia
-			ixx="51563.7946245021"
-			ixy="0.552841467322453"
-			ixz="-212.267889356987"
-			iyy="49495.9076886951"
-			iyz="1.80688027777408"
-			izz="54368.3241585813" />
-		    </inertial>
 		    <visual>
 		      <origin
@@ -199,18 +129,4 @@
 		  </link>
 		  <link name="${prefix}link_5">
-		    <inertial>
-		      <origin
-			xyz="-0.856906936709003 0.000456131051686355 -0.857257705801685"
-			rpy="0 0 0" />
-		      <mass
-			value="48654.354928172" />
-		      <inertia
-			ixx="51563.7946245021"
-			ixy="0.552841467322453"
-			ixz="-212.267889356987"
-			iyy="49495.9076886951"
-			iyz="1.80688027777408"
-			izz="54368.3241585813" />
-		    </inertial>
 		    <visual>
 		      <origin
@@ -238,18 +154,4 @@
 		  </link>
 		  <link name="${prefix}link_6">
-		    <inertial>
-		      <origin
-			xyz="-0.957051849301239 0.000456131051686355 -0.857390019418947"
-			rpy="0 0 0" />
-		      <mass
-			value="48654.354928172" />
-		      <inertia
-			ixx="51563.7946245021"
-			ixy="0.552841467322453"
-			ixz="-212.267889356987"
-			iyy="49495.9076886951"
-			iyz="1.80688027777408"
-			izz="54368.3241585813" />
-		    </inertial>
 		    <visual>
 		      <origin
@@ -276,9 +178,9 @@
 		    </collision>
 		  </link>
-        	  <link name="${prefix}tool0"/>
+          <link name="${prefix}tool0"/>
 	<!-- joints -->
 		  <joint name="${prefix}joint_1" type="revolute">
 		    <origin
-		      xyz="0 0 0.24477"
+		      xyz="0 0 0.245"
 		      rpy="0 0 0" />
 		    <parent
@@ -292,16 +194,5 @@
 		      upper="2.967"
 		      effort="0"
-		      velocity="2.8" />
-		    <calibration
-		      rising="0"
-		      falling="0" />
-		    <dynamics
-		      damping="0"
-		      friction="0" />
-		    <!--safety_controller
-		      soft_lower_limit="0"
-		      soft_upper_limit="0"
-		      k_position="0"
-		      k_velocity="0" /-->
+		      velocity="2.879" />
 		  </joint>
 		  <joint name="${prefix}joint_2" type="revolute">
@@ -319,20 +210,9 @@
 		      upper="2.78"
 		      effort="0"
-		      velocity="2.8" />
-		    <calibration
-		      rising="0"
-		      falling="0" />
-		    <dynamics
-		      damping="0"
-		      friction="0" />
-		    <!--safety_controller
-		      soft_lower_limit="0"
-		      soft_upper_limit="0"
-		      k_position="0"
-		      k_velocity="0" /-->
+		      velocity="2.879" />
 		  </joint>
 		  <joint name="${prefix}joint_3" type="revolute">
 		    <origin
-		      xyz="0 -0.18815 0.77"
+		      xyz="0 -0.18759 0.77"
 		      rpy="0 0 0" />
 		    <parent
@@ -343,23 +223,12 @@
 		      xyz="0 -1 0" />
 		    <limit
-		      lower="4.08"
+		      lower="-4.08"
 		      upper="1.38"
 		      effort="0"
-		      velocity="3.0" />
-		    <calibration
-		      rising="0"
-		      falling="0" />
-		    <dynamics
-		      damping="0"
-		      friction="0" />
-		    <!--safety_controller
-		      soft_lower_limit="0"
-		      soft_upper_limit="0"
-		      k_position="0"
-		      k_velocity="0" /-->
+		      velocity="3.054" />
 		  </joint>
 		  <joint name="${prefix}joint_4" type="revolute">
 		    <origin
-		      xyz="0.1847 0 0.1"
+		      xyz="0.18425 0 0.1"
 		      rpy="0 0 0" />
 		    <parent
@@ -373,20 +242,9 @@
 		      upper="3.48"
 		      effort="0"
-		      velocity="6.1" />
-		    <calibration
-		      rising="0"
-		      falling="0" />
-		    <dynamics
-		      damping="0"
-		      friction="0" />
-		    <!--safety_controller
-		      soft_lower_limit="0"
-		      soft_upper_limit="0"
-		      k_position="0"
-		      k_velocity="0" /-->
+		      velocity="6.108" />
 		  </joint>
 		  <joint name="${prefix}joint_5" type="revolute">
 		    <origin
-		      xyz="0.55575 0.00019326 0.00073427"
+		      xyz="0.55575 0 0"
 		      rpy="0 0 0" />
 		    <parent
@@ -400,20 +258,9 @@
 		      upper="2.43"
 		      effort="0"
-		      velocity="5.9" />
-		    <calibration
-		      rising="0"
-		      falling="0" />
-		    <dynamics
-		      damping="0"
-		      friction="0" />
-		    <!--safety_controller
-		      soft_lower_limit="0"
-		      soft_upper_limit="0"
-		      k_position="0"
-		      k_velocity="0" /-->
+		      velocity="5.934" />
 		  </joint>
 		  <joint name="${prefix}joint_6" type="revolute">
 		    <origin
-		      xyz="0.10014 0 0.00013231"
+		      xyz="0.1 0 0"
 		      rpy="0 0 0" />
 		    <parent
@@ -427,16 +274,5 @@
 		      upper="7.84"
 		      effort="0"
-		      velocity="9.0" />
-		    <calibration
-		      rising="0"
-		      falling="0" />
-		    <dynamics
-		      damping="0"
-		      friction="0" />
-		    <!--safety_controller
-		      soft_lower_limit="0"
-		      soft_upper_limit="0"
-		      k_position="0"
-		      k_velocity="0" /-->
+		      velocity="9.075" />
 		  </joint>
 		  <joint name="${prefix}joint_6-tool0" type="fixed">
