Commit message: Fix incorrect J3 joint limits in m430iA2F URDF.
Updated arm_navigation package as well.

File: fanuc_config/urdf/m430ia2f.urdf (robot description, URDF)
Before this commit: robot m430ia2f, 7 links, 6 joints
Joints:
- joint joint_1: limit lower=-3.1415 upper=3.1415 effort=0 velocity=5.23598775598 -> lower=-3.1415 upper=3.1415 effort=0 velocity=5.24
- joint joint_2: limit lower=-2.00707 upper=2.00707 effort=0 velocity=5.58505360638 -> lower=-2.01 upper=2.01 effort=0 velocity=5.59
- joint joint_3: limit lower=-1.771457 upper=1.771457 effort=0 velocity=5.58505360638 -> lower=-3.49 upper=3.49 effort=0 velocity=5.59
- joint joint_4: limit lower=-2.617917 upper=2.617917 effort=0 velocity=6.28318530718 -> lower=-2.62 upper=2.62 effort=0 velocity=6.28
- joint joint_5: limit lower=-4.71225 upper=4.71225 effort=0 velocity=20.9439510239 -> lower=-4.71 upper=4.71 effort=0 velocity=20.94

File: fanuc_config/urdf/m430ia2f_macro.xacro (robot description, xacro)
@@ -112,5 +112,5 @@
 			<child link="${prefix}link_1"/>
 			<axis xyz="0 0 1"/>
-			<limit lower="-3.1415" upper="3.1415" effort="0" velocity="5.23598775598"/>
+			<limit lower="-3.1415" upper="3.1415" effort="0" velocity="5.24"/>
 		</joint>
 		<joint name="${prefix}joint_2" type="revolute">
@@ -119,5 +119,5 @@
 			<child link="${prefix}link_2"/>
 			<axis xyz="0 1 0"/>
-			<limit lower="-2.00707" upper="2.00707" effort="0" velocity="5.58505360638"/>
+			<limit lower="-2.01" upper="2.01" effort="0" velocity="5.59"/>
 		</joint>
 		<joint name="${prefix}joint_3" type="revolute">
@@ -127,5 +127,5 @@
 			<child link="${prefix}link_3"/>
 			<axis xyz="0 1 0"/>
-			<limit lower="-1.771457" upper="1.771457" effort="0" velocity="5.58505360638"/>
+			<limit lower="-3.49" upper="3.49" effort="0" velocity="5.59"/>
 		</joint>
 		<joint name="${prefix}joint_4" type="revolute">
@@ -135,5 +135,5 @@
 			<child link="${prefix}link_4"/>
 			<axis xyz="0 1 0"/>
-			<limit lower="-2.617917" upper="2.617917" effort="0" velocity="6.28318530718"/>
+			<limit lower="-2.62" upper="2.62" effort="0" velocity="6.28"/>
 		</joint>
 		<joint name="${prefix}joint_5" type="revolute">
@@ -142,5 +142,5 @@
 			<child link="${prefix}link_5"/>
 			<axis xyz="0 0 1"/>
-			<limit lower="-4.71225" upper="4.71225" effort="0" velocity="20.9439510239"/>
+			<limit lower="-4.71" upper="4.71" effort="0" velocity="20.94"/>
 		</joint>
 		<joint name="${prefix}joint_5-tool0" type="fixed">

Commit message: Update meshes (collision and visual) and xacro of M-430iA/2F.
Minimal changes: result of the arm_navigation wizard showed no changes for the arm_navigation package.

File: fanuc_config/urdf/m430ia2f.urdf (robot description, URDF)
Before this commit: robot m430ia2f, 7 links, 6 joints
Joints:
- joint joint_1: origin xyz=-6.0758E-19 1.2493E-16 0.44 rpy=0 0 0 -> xyz=0 0 0.44 rpy=0 0 0
- joint joint_2: origin xyz=-1.4097E-17 0.171 -4.4409E-16 rpy=0 0 0 -> xyz=0 0.171 0 rpy=0 0 0
- joint joint_3: limit lower=-3.49 upper=3.49 effort=0 velocity=5.59 -> lower=-3.34 upper=3.34 effort=0 velocity=5.59; origin xyz=1.2197E-19 -0.171 0.350 rpy=0 0 0 -> xyz=0 -0.171 0.35 rpy=0 0 0
- joint joint_4: origin xyz=-2.6075E-17 -0.06 0.55 rpy=0 0 0 -> xyz=0 -0.06 0.55 rpy=0 0 0
- joint joint_5: origin xyz=1.4734E-16 -0.035 0.065 rpy=0 0 0 -> xyz=0 -0.035 0.065 rpy=0 0 0

File: fanuc_config/urdf/m430ia2f_macro.xacro (robot description, xacro)
@@ -10,5 +10,5 @@
 				</geometry>
 				<material name="white">
-					<color rgba="1 1 1 1"/>
+					<color rgba="0.9 0.9 0.9 1"/>
 				</material>
 			</visual>
@@ -56,4 +56,8 @@
 		<link name="${prefix}link_3">
 			<visual>
+				<!-- coordinate origin for link_3 is not at mate centre, -->
+				<!-- so compensate (53mm dZ between link_3-link_2 mate -->
+				<!-- and coordinate origin) -->
+				<!-- origin xyz="0 0 0" rpy="0 0 0"/ -->
 				<origin xyz="0 0 0.053" rpy="0 0 0"/>
 				<geometry>
@@ -65,4 +69,6 @@
 			</visual>
 			<collision>
+				<!-- see earlier comment -->
+				<!-- origin xyz="0 0 0" rpy="0 0 0"/ -->
 				<origin xyz="0 0 0.053" rpy="0 0 0"/>
 				<geometry>
@@ -108,5 +114,5 @@
 		<!-- joints -->
 		<joint name="${prefix}joint_1" type="revolute">
-			<origin xyz="-6.0758E-19 1.2493E-16 0.44" rpy="0 0 0"/>
+			<origin xyz="0 0 0.44" rpy="0 0 0"/>
 			<parent link="${prefix}base_link"/>
 			<child link="${prefix}link_1"/>
@@ -115,5 +121,5 @@
 		</joint>
 		<joint name="${prefix}joint_2" type="revolute">
-			<origin xyz="-1.4097E-17 0.171 -4.4409E-16" rpy="0 0 0"/>
+			<origin xyz="0 0.171 0" rpy="0 0 0"/>
 			<parent link="${prefix}link_1"/>
 			<child link="${prefix}link_2"/>
@@ -122,14 +128,16 @@
 		</joint>
 		<joint name="${prefix}joint_3" type="revolute">
-			<!-- origin xyz="1.2197E-19 -0.171 0.403" rpy="0 0 0" / -->
-			<origin xyz="1.2197E-19 -0.171 0.350" rpy="0 0 0"/>
+			<!-- see earlier comment -->
+			<!-- origin xyz="0 -0.171 0.403" rpy="0 0 0"/ -->
+			<origin xyz="0 -0.171 0.35" rpy="0 0 0"/>
 			<parent link="${prefix}link_2"/>
 			<child link="${prefix}link_3"/>
 			<axis xyz="0 1 0"/>
-			<limit lower="-3.49" upper="3.49" effort="0" velocity="5.59"/>
+			<limit lower="-3.34" upper="3.34" effort="0" velocity="5.59"/>
 		</joint>
 		<joint name="${prefix}joint_4" type="revolute">
-			<!-- origin xyz="-2.6075E-17 -0.06 0.497" rpy="0 0 0" / -->
-			<origin xyz="-2.6075E-17 -0.06 0.55" rpy="0 0 0"/>
+			<!-- see earlier comment -->
+			<!-- origin xyz="0 -0.06 0.497" rpy="0 0 0"/ -->
+			<origin xyz="0 -0.06 0.55" rpy="0 0 0"/>
 			<parent link="${prefix}link_3"/>
 			<child link="${prefix}link_4"/>
@@ -138,5 +146,5 @@
 		</joint>
 		<joint name="${prefix}joint_5" type="revolute">
-			<origin xyz="1.4734E-16 -0.035 0.065" rpy="0 0 0"/>
+			<origin xyz="0 -0.035 0.065" rpy="0 0 0"/>
 			<parent link="${prefix}link_4"/>
 			<child link="${prefix}link_5"/>
