Commit message: Fix max joint velocity for J1 in LR Mate 200iC/5H.

File: fanuc_config/urdf/lrmate200ic5h.urdf (robot description, URDF)
Before this commit: robot lrmate200ic5h, 7 links, 6 joints
Joints:
- joint joint_1: limit lower=-2.965 upper=2.965 effort=0 velocity=5.93 -> lower=-2.965 upper=2.965 effort=0 velocity=6.11

File: fanuc_config/urdf/lrmate200ic5h_macro.xacro (robot description, xacro)
@@ -104,5 +104,5 @@
 			<child link="${prefix}link_1" />
 			<axis xyz="0 0 1" />
-			<limit lower="-2.965" upper="2.965" effort="0" velocity="5.93" />
+			<limit lower="-2.965" upper="2.965" effort="0" velocity="6.11" />
 		</joint>
 		<joint name="${prefix}joint_2" type="revolute">
