Commit message: Fix formatting of URDFs and improve appearance of robot models in RVIZ (use proper colours where possible).

File: fanuc_config/urdf/m10ia_macro.xacro (robot description, xacro)
@@ -1,323 +1,160 @@
-<?xml version="1.0" ?>
+<?xml version="1.0"?>
 <robot xmlns:xacro="http://ros.org/wiki/xacro">
 	<xacro:macro name="m10ia" params="prefix">
-		<!-- link list -->
+		<!-- links -->
 		<link name="${prefix}base_link">
 			<visual>
-     			<origin
-        		xyz="0 0 0"
-       			rpy="-1.578 0 0" />
-      			<geometry>
-        			<mesh
-          			filename="package://fanuc_config/meshes/m10ia/visual/base_link.stl" />
-      			</geometry>
-      			<material
-        			name="grey">
-        			<color
-          			rgba="0.75 0.75 0.75 1" />
-      			</material>
-    		</visual>
- 			<collision>
-     			<origin
-        		xyz="0 0 0"
-       			rpy="-1.578 0 0" />
+				<origin xyz="0 0 0" rpy="-1.578 0 0"/>
 				<geometry>
-					<mesh filename="package://fanuc_config/meshes/m10ia/collision/base_link.stl" />
+					<mesh filename="package://fanuc_config/meshes/m10ia/visual/base_link.stl"/>
 				</geometry>
-				<material name="yellow">
-					<color rgba="1 1 0 1"/>
+				<material name="fgrey">
+					<color rgba="0.20 0.20 0.20 1"/>
 				</material>
+			</visual>
+			<collision>
+				<origin xyz="0 0 0" rpy="-1.578 0 0"/>
+				<geometry>
+					<mesh filename="package://fanuc_config/meshes/m10ia/collision/base_link.stl"/>
+				</geometry>
 			</collision>
 		</link>
 		<link name="${prefix}link_1">
 			<visual>
-      			<origin
-        			xyz="0 0 0"
-        			rpy="0 0 0" />
-      			<geometry>
-        			<mesh
-          			filename="package://fanuc_config/meshes/m10ia/visual/link_1.stl" />
-      			</geometry>
-      			<material name="grey"/>
-    		</visual>
+				<origin xyz="0 0 0" rpy="0 0 0"/>
+				<geometry>
+					<mesh filename="package://fanuc_config/meshes/m10ia/visual/link_1.stl"/>
+				</geometry>
+				<material name="fyel">
+					<color rgba="0.9 0.9 0 1"/>
+				</material>
+			</visual>
 			<collision>
-      			<origin
-        			xyz="0 0 0"
-        			rpy="0 0 0" />
+				<origin xyz="0 0 0" rpy="0 0 0"/>
 				<geometry>
-					<mesh filename="package://fanuc_config/meshes/m10ia/collision/link_1.stl" />
+					<mesh filename="package://fanuc_config/meshes/m10ia/collision/link_1.stl"/>
 				</geometry>
-				<material name="yellow"/>
 			</collision>
 		</link>
 		<link name="${prefix}link_2">
-		    <visual>
-      			<origin
-        			xyz="0 0 0"
-        			rpy="0 0 0" />
-      			<geometry>
-        			<mesh
-          			filename="package://fanuc_config/meshes/m10ia/visual/link_2.stl" />
-      			</geometry>
-      			<material name="grey"/>
-    		</visual>
+			<visual>
+				<origin xyz="0 0 0" rpy="0 0 0"/>
+				<geometry>
+					<mesh filename="package://fanuc_config/meshes/m10ia/visual/link_2.stl"/>
+				</geometry>
+				<material name="fyel"/>
+			</visual>
 			<collision>
-      			<origin
-        			xyz="0 0 0"
-        			rpy="0 0 0" />
+				<origin xyz="0 0 0" rpy="0 0 0"/>
 				<geometry>
-					<mesh filename="package://fanuc_config/meshes/m10ia/collision/link_2.stl" />
+					<mesh filename="package://fanuc_config/meshes/m10ia/collision/link_2.stl"/>
 				</geometry>
-				<material name="yellow"/>
 			</collision>
 		</link>
 		<link name="${prefix}link_3">
 			<visual>
-				<origin
-					xyz="0 0 0"
-					rpy="0 0 0" />
-			  	<geometry>
-					<mesh
-				  	filename="package://fanuc_config/meshes/m10ia/visual/link_3.stl" />
-			  	</geometry>
-			  	<material name="grey"/>
+				<origin xyz="0 0 0" rpy="0 0 0"/>
+				<geometry>
+					<mesh filename="package://fanuc_config/meshes/m10ia/visual/link_3.stl"/>
+				</geometry>
+				<material name="fyel"/>
 			</visual>
 			<collision>
-      			<origin
-        			xyz="0 0 0"
-        			rpy="0 0 0" />
+				<origin xyz="0 0 0" rpy="0 0 0"/>
 				<geometry>
-					<mesh filename="package://fanuc_config/meshes/m10ia/collision/link_3.stl" />
+					<mesh filename="package://fanuc_config/meshes/m10ia/collision/link_3.stl"/>
 				</geometry>
-				<material name="yellow"/>
 			</collision>
 		</link>
 		<link name="${prefix}link_4">
 			<visual>
-				  <origin
-					xyz="0 0 0"
-					rpy="0 0 0" />
-				  <geometry>
-					<mesh
-					  filename="package://fanuc_config/meshes/m10ia/visual/link_4.stl" />
-				  </geometry>
-				  <material name="grey"/>
+				<origin xyz="0 0 0" rpy="0 0 0"/>
+				<geometry>
+					<mesh filename="package://fanuc_config/meshes/m10ia/visual/link_4.stl"/>
+				</geometry>
+				<material name="fyel"/>
 			</visual>
 			<collision>
-      			<origin
-        			xyz="0 0 0"
-        			rpy="0 0 0" />
+				<origin xyz="0 0 0" rpy="0 0 0"/>
 				<geometry>
-					<mesh filename="package://fanuc_config/meshes/m10ia/collision/link_4.stl" />
+					<mesh filename="package://fanuc_config/meshes/m10ia/collision/link_4.stl"/>
 				</geometry>
-				<material name="yellow"/>
 			</collision>
 		</link>
 		<link name="${prefix}link_5">
 			<visual>
-				<origin
-					xyz="0 0 0"
-					rpy="0 0 0" />
+				<origin xyz="0 0 0" rpy="0 0 0"/>
 				<geometry>
-					<mesh
-					  filename="package://fanuc_config/meshes/m10ia/visual/link_5.stl" />
+					<mesh filename="package://fanuc_config/meshes/m10ia/visual/link_5.stl"/>
 				</geometry>
-				<material name="grey"/>
+				<material name="fyel"/>
 			</visual>
 			<collision>
-      			<origin
-        			xyz="0 0 0"
-        			rpy="0 0 0" />
+				<origin xyz="0 0 0" rpy="0 0 0"/>
 				<geometry>
-					<mesh filename="package://fanuc_config/meshes/m10ia/collision/link_5.stl" />
+					<mesh filename="package://fanuc_config/meshes/m10ia/collision/link_5.stl"/>
 				</geometry>
-				<material name="yellow"/>
 			</collision>
 		</link>
 		<link name="${prefix}link_6">
 			<visual>
-				<origin
-					xyz="0 0 0"
-					rpy="0 0 0" />
+				<origin xyz="0 0 0" rpy="0 0 0"/>
 				<geometry>
-					<mesh
-					  filename="package://fanuc_config/meshes/m10ia/visual/link_6.stl" />
+					<mesh filename="package://fanuc_config/meshes/m10ia/visual/link_6.stl"/>
 				</geometry>
-				<material name="grey"/>
+				<material name="fblack">
+					<color rgba="0.1 0.1 0.1 1"/>
+				</material>
 			</visual>
 			<collision>
-      			<origin
-        			xyz="0 0 0"
-        			rpy="0 0 0" />
+				<origin xyz="0 0 0" rpy="0 0 0"/>
 				<geometry>
-					<mesh filename="package://fanuc_config/meshes/m10ia/collision/link_6.stl" />
+					<mesh filename="package://fanuc_config/meshes/m10ia/collision/link_6.stl"/>
 				</geometry>
-				<material name="yellow"/>
 			</collision>
 		</link>
 		<link name="${prefix}tool0"/>
-		<!-- end of link list -->
-		<!-- joint list -->
+		<!-- joints -->
 		<joint name="${prefix}joint_1" type="revolute">
-			<origin
-      			xyz="0 0 0"
-      			rpy="0 0 0" />
-			<parent
-			  link="base_link" />
-			<child
-			  link="link_1" />
-			<axis
-			  xyz="0 0 1" />
-			<limit
-			  lower="-5.93"
-			  upper="5.93"
-			  effort="0"
-			  velocity="3.665" />
-			<calibration
-			  rising="0"
-			  falling="0" />
-			<dynamics
-			  damping="0"
-			  friction="0" />
-<!--			<safety_controller
-			  soft_lower_limit="0"
-			  soft_upper_limit="0"
-			  k_position="0"
-			  k_velocity="0" /> -->
+			<origin xyz="0 0 0" rpy="0 0 0"/>
+			<parent link="base_link"/>
+			<child link="link_1"/>
+			<axis xyz="0 0 1"/>
+			<limit lower="-5.93" upper="5.93" effort="0" velocity="3.665"/>
 		</joint>
 		<joint name="${prefix}joint_2" type="revolute">
-			<origin
-			  xyz="0.15 -0.04 0.45"
-      		  rpy="0 0 0" />
-			<parent
-			  link="link_1" />
-			<child
-			  link="link_2" />
-			<axis
-			  xyz="0 1 0" />
-			<limit
-			  lower="-4.36"
-			  upper="4.36"
-			  effort="0"
-			  velocity="3.32" />
-			<calibration
-			  rising="0"
-			  falling="0" />
-			<dynamics
-			  damping="0"
-			  friction="0" />
-<!--			<safety_controller
-			  soft_lower_limit="0"
-			  soft_upper_limit="0"
-			  k_position="0"
-			  k_velocity="0" /> -->
-  		</joint>
+			<origin xyz="0.15 -0.04 0.45" rpy="0 0 0"/>
+			<parent link="link_1"/>
+			<child link="link_2"/>
+			<axis xyz="0 1 0"/>
+			<limit lower="-4.36" upper="4.36" effort="0" velocity="3.32"/>
+		</joint>
 		<joint name="${prefix}joint_3" type="revolute">
-			<origin
-			  xyz="0 -0.0225 0.6"
-    		  rpy="0 0 0" />
-			<parent
-			  link="link_2" />
-			<child
-			  link="link_3" />
-			<axis
-			  xyz="0 1 0" />
-			<limit
-			  lower="-5.06"
-			  upper="5.06"
-			  effort="0"
-			  velocity="3.665" />
-			<calibration
-			  rising="0"
-			  falling="0" />
-			<dynamics
-			  damping="0"
-			  friction="0" />
-<!--			<safety_controller
-			  soft_lower_limit="0"
-			  soft_upper_limit="0"
-			  k_position="0"
-			  k_velocity="0" /> -->
+			<origin xyz="0 -0.0225 0.6" rpy="0 0 0"/>
+			<parent link="link_2"/>
+			<child link="link_3"/>
+			<axis xyz="0 1 0"/>
+			<limit lower="-5.06" upper="5.06" effort="0" velocity="3.665"/>
 		</joint>
 		<joint name="${prefix}joint_4" type="revolute">
-			<origin
-			  xyz="0.1805 0.0625 0.2"
-    		  rpy="0 0 0" />
-			<parent
-			  link="link_3" />
-			<child
-			  link="link_4" />
-			<axis
-			  xyz="1 0 0" />
-			<limit
-			  lower="-6.63"
-			  upper="6.63"
-			  effort="0"
-			  velocity="6.98" />
-			<calibration
-			  rising="0"
-			  falling="0" />
-			<dynamics
-			  damping="0"
-			  friction="0" />
-<!--			<safety_controller
-			  soft_lower_limit="0"
-			  soft_upper_limit="0"
-			  k_position="0"
-			  k_velocity="0" /> -->
+			<origin xyz="0.1805 0.0625 0.2" rpy="0 0 0"/>
+			<parent link="link_3"/>
+			<child link="link_4"/>
+			<axis xyz="1 0 0"/>
+			<limit lower="-6.63" upper="6.63" effort="0" velocity="6.98"/>
 		</joint>
 		<joint name="${prefix}joint_5" type="revolute">
-			<origin
-			  xyz="0.4595 -0.0565 0"
-      		  rpy="0 0 0" />
-			<parent
-			  link="link_4" />
-			<child
-			  link="link_5" />
-			<axis
-			  xyz="0 1 0" />
-			<limit
-			  lower="-6.63"
-			  upper="6.63"
-			  effort="0"
-			  velocity="3.98" />
-			<calibration
-			  rising="0"
-			  falling="0" />
-			<dynamics
-			  damping="0"
-			  friction="0" />
-<!--			<safety_controller
-			  soft_lower_limit="0"
-			  soft_upper_limit="0"
-			  k_position="0"
-			  k_velocity="0" /> -->
+			<origin xyz="0.4595 -0.0565 0" rpy="0 0 0"/>
+			<parent link="link_4"/>
+			<child link="link_5"/>
+			<axis xyz="0 1 0"/>
+			<limit lower="-6.63" upper="6.63" effort="0" velocity="3.98"/>
 		</joint>
 		<joint name="${prefix}joint_6" type="revolute">
-			<origin
-			  xyz="0.1 0.0565 0"
-    		  rpy="0 0 0" />
-			<parent
-			  link="link_5" />
-			<child
-			  link="link_6" />
-			<axis
-			  xyz="1 0 0" />
-			<limit
-			  lower="-12.566"
-			  upper="12.566"
-			  effort="0"
-			  velocity="10.47" />
-			<calibration
-			  rising="0"
-			  falling="0" />
-			<dynamics
-			  damping="0"
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
File: fanuc_config/urdf/m16ib20_macro.xacro (robot description, xacro)
@@ -2,283 +2,163 @@
 <robot xmlns:xacro="http://ros.org/wiki/xacro">
 	<xacro:macro name="m16ib20" params="prefix">
-	<!-- links -->
-		  <link name="${prefix}base_link">
-		    <visual>
-		      <origin
-			xyz="0 0 0"
-			rpy="0 0 0" />
-		      <geometry>
-			<mesh
-			  filename="package://fanuc_config/meshes/m16ib20/visual/base_link.STL" />
-		      </geometry>
-		      <material
-			name="">
-			<color
-			  rgba="1 1 0 1" />
-		      </material>
-		    </visual>
-		    <collision>
-		      <origin
-			xyz="0 0 0"
-			rpy="0 0 0" />
-		      <geometry>
-			<mesh
-			  filename="package://fanuc_config/meshes/m16ib20/collision/base_link.STL" />
-		      </geometry>
-		    </collision>
-		  </link>
-		  <link name="${prefix}link_1">
-		    <visual>
-		      <origin
-			xyz="0 0 0"
-			rpy="0 0 0" />
-		      <geometry>
-			<mesh
-			  filename="package://fanuc_config/meshes/m16ib20/visual/Link_1.STL" />
-		      </geometry>
-		      <material
-			name="">
-			<color
-			  rgba="1 1 0 1" />
-		      </material>
-		    </visual>
-		    <collision>
-		      <origin
-			xyz="0 0 0"
-			rpy="0 0 0" />
-		      <geometry>
-			<mesh
-			  filename="package://fanuc_config/meshes/m16ib20/collision/Link_1.STL" />
-		      </geometry>
-		    </collision>
-		  </link>
-		  <link name="${prefix}link_2">
-		    <visual>
-		      <origin
-			xyz="0 0 0"
-			rpy="0 0 0" />
-		      <geometry>
-			<mesh
-			  filename="package://fanuc_config/meshes/m16ib20/visual/Link_2.STL" />
-		      </geometry>
-		      <material
-			name="">
-			<color
-			  rgba="1 1 0 1" />
-		      </material>
-		    </visual>
-		    <collision>
-		      <origin
-			xyz="0 0 0"
-			rpy="0 0 0" />
-		      <geometry>
-			<mesh
-			  filename="package://fanuc_config/meshes/m16ib20/collision/Link_2.STL" />
-		      </geometry>
-		    </collision>
-		  </link>
-		  <link name="${prefix}link_3">
-		    <visual>
-		      <origin
-			xyz="0 0 0"
-			rpy="0 0 0" />
-		      <geometry>
-			<mesh
-			  filename="package://fanuc_config/meshes/m16ib20/visual/Link_3.STL" />
-		      </geometry>
-		      <material
-			name="">
-			<color
-			  rgba="1 1 0 1" />
-		      </material>
-		    </visual>
-		    <collision>
-		      <origin
-			xyz="0 0 0"
-			rpy="0 0 0" />
-		      <geometry>
-			<mesh
-			  filename="package://fanuc_config/meshes/m16ib20/collision/Link_3.STL" />
-		      </geometry>
-		    </collision>
-		  </link>
-		  <link name="${prefix}link_4">
-		    <visual>
-		      <origin
-			xyz="0 0 0"
-			rpy="0 0 0" />
-		      <geometry>
-			<mesh
-			  filename="package://fanuc_config/meshes/m16ib20/visual/Link_4.STL" />
-		      </geometry>
-		      <material
-			name="">
-			<color
-			  rgba="1 1 0 1" />
-		      </material>
-		    </visual>
-		    <collision>
-		      <origin
-			xyz="0 0 0"
-			rpy="0 0 0" />
-		      <geometry>
-			<mesh
-			  filename="package://fanuc_config/meshes/m16ib20/collision/Link_4.STL" />
-		      </geometry>
-		    </collision>
-		  </link>
-		  <link name="${prefix}link_5">
-		    <visual>
-		      <origin
-			xyz="0 0 0"
-			rpy="0 0 0" />
-		      <geometry>
-			<mesh
-			  filename="package://fanuc_config/meshes/m16ib20/visual/Link_5.STL" />
-		      </geometry>
-		      <material
-			name="">
-			<color
-			  rgba="1 1 0 1" />
-		      </material>
-		    </visual>
-		    <collision>
-		      <origin
-			xyz="0 0 0"
-			rpy="0 0 0" />
-		      <geometry>
-			<mesh
-			  filename="package://fanuc_config/meshes/m16ib20/collision/Link_5.STL" />
-		      </geometry>
-		    </collision>
-		  </link>
-		  <link name="${prefix}link_6">
-		    <visual>
-		      <origin
-			xyz="0 0 0"
-			rpy="0 0 0" />
-		      <geometry>
-			<mesh
-			  filename="package://fanuc_config/meshes/m16ib20/visual/Link_6.STL" />
-		      </geometry>
-		      <material
-			name="">
-			<color
-			  rgba="1 1 0 1" />
-		      </material>
-		    </visual>
-		    <collision>
-		      <origin
-			xyz="0 0 0"
-			rpy="0 0 0" />
-		      <geometry>
-			<mesh
-			  filename="package://fanuc_config/meshes/m16ib20/collision/Link_6.STL" />
-		      </geometry>
-		    </collision>
-		  </link>
-          <link name="${prefix}tool0"/>
-	<!-- joints -->
-		  <joint name="${prefix}joint_1" type="revolute">
-		    <origin
-		      xyz="0 0 0.245"
-		      rpy="0 0 0" />
-		    <parent
-		      link="base_link" />
-		    <child
-		      link="link_1" />
-		    <axis
-		      xyz="0 0 1" />
-		    <limit
-		      lower="-2.967"
-		      upper="2.967"
-		      effort="0"
-		      velocity="2.879" />
-		  </joint>
-		  <joint name="${prefix}joint_2" type="revolute">
-		    <origin
-		      xyz="0.15 0.18759 0.28"
-		      rpy="0 0 0" />
-		    <parent
-		      link="link_1" />
-		    <child
-		      link="link_2" />
-		    <axis
-		      xyz="0 1 0" />
-		    <limit
-		      lower="-1.38"
-		      upper="2.78"
-		      effort="0"
-		      velocity="2.879" />
-		  </joint>
-		  <joint name="${prefix}joint_3" type="revolute">
-		    <origin
-		      xyz="0 -0.18759 0.77"
-		      rpy="0 0 0" />
-		    <parent
-		      link="link_2" />
-		    <child
-		      link="link_3" />
-		    <axis
-		      xyz="0 -1 0" />
-		    <limit
-		      lower="-4.08"
-		      upper="1.38"
-		      effort="0"
-		      velocity="3.054" />
-		  </joint>
-		  <joint name="${prefix}joint_4" type="revolute">
-		    <origin
-		      xyz="0.18425 0 0.1"
-		      rpy="0 0 0" />
-		    <parent
-		      link="link_3" />
-		    <child
-		      link="link_4" />
-		    <axis
-		      xyz="-1 0 0" />
-		    <limit
-		      lower="-3.48"
-		      upper="3.48"
-		      effort="0"
-		      velocity="6.108" />
-		  </joint>
-		  <joint name="${prefix}joint_5" type="revolute">
-		    <origin
-		      xyz="0.55575 0 0"
-		      rpy="0 0 0" />
-		    <parent
-		      link="link_4" />
-		    <child
-		      link="link_5" />
-		    <axis
-		      xyz="0 -1 0" />
-		    <limit
-		      lower="-2.43"
-		      upper="2.43"
-		      effort="0"
-		      velocity="5.934" />
-		  </joint>
-		  <joint name="${prefix}joint_6" type="revolute">
-		    <origin
-		      xyz="0.1 0 0"
-		      rpy="0 0 0" />
-		    <parent
-		      link="link_5" />
-		    <child
-		      link="link_6" />
-		    <axis
-		      xyz="-1 0 0" />
-		    <limit
-		      lower="-7.84"
-		      upper="7.84"
-		      effort="0"
-		      velocity="9.075" />
-		  </joint>
-		  <joint name="${prefix}joint_6-tool0" type="fixed">
-		      <parent link="${prefix}link_6"/>
-	              <child link="${prefix}tool0"/>
-          	      <origin xyz="0 0 0" rpy="0 0 0"/>
-	          </joint>
+		<!-- links -->
+		<link name="${prefix}base_link">
+			<visual>
+				<origin xyz="0 0 0" rpy="0 0 0"/>
+				<geometry>
+					<mesh filename="package://fanuc_config/meshes/m16ib20/visual/base_link.STL"/>
+				</geometry>
+				<material name="fyel">
+					<color rgba="0.9 0.9 0 1" />
+				</material>
+			</visual>
+			<collision>
+				<origin xyz="0 0 0" rpy="0 0 0"/>
+				<geometry>
+					<mesh filename="package://fanuc_config/meshes/m16ib20/collision/base_link.STL"/>
+				</geometry>
+			</collision>
+		</link>
+		<link name="${prefix}link_1">
+			<visual>
+				<origin xyz="0 0 0" rpy="0 0 0"/>
+				<geometry>
+					<mesh filename="package://fanuc_config/meshes/m16ib20/visual/Link_1.STL"/>
+				</geometry>
+				<material name="fyel" />
+			</visual>
+			<collision>
+				<origin xyz="0 0 0" rpy="0 0 0"/>
+				<geometry>
+					<mesh filename="package://fanuc_config/meshes/m16ib20/collision/Link_1.STL"/>
+				</geometry>
+			</collision>
+		</link>
+		<link name="${prefix}link_2">
+			<visual>
+				<origin xyz="0 0 0" rpy="0 0 0"/>
+				<geometry>
+					<mesh filename="package://fanuc_config/meshes/m16ib20/visual/Link_2.STL"/>
+				</geometry>
+				<material name="fyel" />
+			</visual>
+			<collision>
+				<origin xyz="0 0 0" rpy="0 0 0"/>
+				<geometry>
+					<mesh filename="package://fanuc_config/meshes/m16ib20/collision/Link_2.STL"/>
+				</geometry>
+			</collision>
+		</link>
+		<link name="${prefix}link_3">
+			<visual>
+				<origin xyz="0 0 0" rpy="0 0 0"/>
+				<geometry>
+					<mesh filename="package://fanuc_config/meshes/m16ib20/visual/Link_3.STL"/>
+				</geometry>
+				<material name="fyel" />
+			</visual>
+			<collision>
+				<origin xyz="0 0 0" rpy="0 0 0"/>
+				<geometry>
+					<mesh filename="package://fanuc_config/meshes/m16ib20/collision/Link_3.STL"/>
+				</geometry>
+			</collision>
+		</link>
+		<link name="${prefix}link_4">
+			<visual>
+				<origin xyz="0 0 0" rpy="0 0 0"/>
+				<geometry>
+					<mesh filename="package://fanuc_config/meshes/m16ib20/visual/Link_4.STL"/>
+				</geometry>
+				<material name="fyel" />
+			</visual>
+			<collision>
+				<origin xyz="0 0 0" rpy="0 0 0"/>
+				<geometry>
+					<mesh filename="package://fanuc_config/meshes/m16ib20/collision/Link_4.STL"/>
+				</geometry>
+			</collision>
+		</link>
+		<link name="${prefix}link_5">
+			<visual>
+				<origin xyz="0 0 0" rpy="0 0 0"/>
+				<geometry>
+					<mesh filename="package://fanuc_config/meshes/m16ib20/visual/Link_5.STL"/>
+				</geometry>
+				<material name="fyel" />
+			</visual>
+			<collision>
+				<origin xyz="0 0 0" rpy="0 0 0"/>
+				<geometry>
+					<mesh filename="package://fanuc_config/meshes/m16ib20/collision/Link_5.STL"/>
+				</geometry>
+			</collision>
+		</link>
+		<link name="${prefix}link_6">
+			<visual>
+				<origin xyz="0 0 0" rpy="0 0 0"/>
+				<geometry>
+					<mesh filename="package://fanuc_config/meshes/m16ib20/visual/Link_6.STL"/>
+				</geometry>
+				<material name="fblack">
+					<color rgba="0.1 0.1 0.1 1"/>
+				</material>
+			</visual>
+			<collision>
+				<origin xyz="0 0 0" rpy="0 0 0"/>
+				<geometry>
+					<mesh filename="package://fanuc_config/meshes/m16ib20/collision/Link_6.STL"/>
+				</geometry>
+			</collision>
+		</link>
+		<link name="${prefix}tool0"/>
+		<!-- joints -->
+		<joint name="${prefix}joint_1" type="revolute">
+			<origin xyz="0 0 0.245" rpy="0 0 0"/>
+			<parent link="base_link"/>
+			<child link="link_1"/>
+			<axis xyz="0 0 1"/>
+			<limit lower="-2.967" upper="2.967" effort="0" velocity="2.879"/>
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