Commit message: Fix formatting of URDFs and improve appearance of robot models in RVIZ (use proper colours where possible).

File: fanuc_config/urdf/m430ia2f_macro.xacro (robot description, xacro)
@@ -1,20 +1,20 @@
-<?xml version="1.0" ?>
+<?xml version="1.0"?>
 <robot xmlns:xacro="http://ros.org/wiki/xacro">
-    <xacro:macro name="m430ia2f" params="prefix">
-        <!-- links -->
+	<xacro:macro name="m430ia2f" params="prefix">
+		<!-- links -->
 		<link name="${prefix}base_link">
 			<visual>
-				<origin xyz="0 0 0" rpy="0 0 0" />
+				<origin xyz="0 0 0" rpy="0 0 0"/>
 				<geometry>
-					<mesh filename="package://fanuc_config/meshes/m430ia2f/visual/base_link.stl" />
+					<mesh filename="package://fanuc_config/meshes/m430ia2f/visual/base_link.stl"/>
 				</geometry>
 				<material name="white">
-					<color rgba="1 1 1 1" />
+					<color rgba="1 1 1 1"/>
 				</material>
 			</visual>
 			<collision>
-				<origin xyz="0 0 0" rpy="0 0 0" />
+				<origin xyz="0 0 0" rpy="0 0 0"/>
 				<geometry>
-					<mesh filename="package://fanuc_config/meshes/m430ia2f/collision/base_link.stl" />
+					<mesh filename="package://fanuc_config/meshes/m430ia2f/collision/base_link.stl"/>
 				</geometry>
 			</collision>
@@ -22,16 +22,16 @@
 		<link name="${prefix}link_1">
 			<visual>
-				<origin xyz="0 0 0" rpy="0 0 0" />
+				<origin xyz="0 0 0" rpy="0 0 0"/>
 				<geometry>
-					<mesh filename="package://fanuc_config/meshes/m430ia2f/visual/link_1.stl" />
+					<mesh filename="package://fanuc_config/meshes/m430ia2f/visual/link_1.stl"/>
 				</geometry>
 				<material name="">
-					<color rgba="0.89804 0.89804 0.89804 1" />
+					<color rgba="0.89804 0.89804 0.89804 1"/>
 				</material>
 			</visual>
 			<collision>
-				<origin xyz="0 0 0" rpy="0 0 0" />
+				<origin xyz="0 0 0" rpy="0 0 0"/>
 				<geometry>
-					<mesh filename="package://fanuc_config/meshes/m430ia2f/collision/link_1.stl" />
+					<mesh filename="package://fanuc_config/meshes/m430ia2f/collision/link_1.stl"/>
 				</geometry>
 			</collision>
@@ -39,16 +39,16 @@
 		<link name="${prefix}link_2">
 			<visual>
-				<origin xyz="0 0 0" rpy="0 0 0" />
+				<origin xyz="0 0 0" rpy="0 0 0"/>
 				<geometry>
-					<mesh filename="package://fanuc_config/meshes/m430ia2f/visual/link_2.stl" />
+					<mesh filename="package://fanuc_config/meshes/m430ia2f/visual/link_2.stl"/>
 				</geometry>
 				<material name="">
-					<color rgba="0.89804 0.89804 0.89804 1" />
+					<color rgba="0.89804 0.89804 0.89804 1"/>
 				</material>
 			</visual>
 			<collision>
-				<origin xyz="0 0 0" rpy="0 0 0" />
+				<origin xyz="0 0 0" rpy="0 0 0"/>
 				<geometry>
-					<mesh filename="package://fanuc_config/meshes/m430ia2f/collision/link_2.stl" />
+					<mesh filename="package://fanuc_config/meshes/m430ia2f/collision/link_2.stl"/>
 				</geometry>
 			</collision>
@@ -56,16 +56,16 @@
 		<link name="${prefix}link_3">
 			<visual>
-				<origin xyz="0 0 0.053" rpy="0 0 0" />
+				<origin xyz="0 0 0.053" rpy="0 0 0"/>
 				<geometry>
-					<mesh filename="package://fanuc_config/meshes/m430ia2f/visual/link_3.stl" />
+					<mesh filename="package://fanuc_config/meshes/m430ia2f/visual/link_3.stl"/>
 				</geometry>
 				<material name="">
-					<color rgba="0.89804 0.89804 0.89804 1" />
+					<color rgba="0.89804 0.89804 0.89804 1"/>
 				</material>
 			</visual>
 			<collision>
-				<origin xyz="0 0 0.053" rpy="0 0 0" />
+				<origin xyz="0 0 0.053" rpy="0 0 0"/>
 				<geometry>
-					<mesh filename="package://fanuc_config/meshes/m430ia2f/collision/link_3.stl" />
+					<mesh filename="package://fanuc_config/meshes/m430ia2f/collision/link_3.stl"/>
 				</geometry>
 			</collision>
@@ -73,16 +73,16 @@
 		<link name="${prefix}link_4">
 			<visual>
-				<origin xyz="0 0 0" rpy="0 0 0" />
+				<origin xyz="0 0 0" rpy="0 0 0"/>
 				<geometry>
-					<mesh filename="package://fanuc_config/meshes/m430ia2f/visual/link_4.stl" />
+					<mesh filename="package://fanuc_config/meshes/m430ia2f/visual/link_4.stl"/>
 				</geometry>
 				<material name="">
-					<color rgba="0.89804 0.89804 0.89804 1" />
+					<color rgba="0.89804 0.89804 0.89804 1"/>
 				</material>
 			</visual>
 			<collision>
-				<origin xyz="0 0 0" rpy="0 0 0" />
+				<origin xyz="0 0 0" rpy="0 0 0"/>
 				<geometry>
-					<mesh filename="package://fanuc_config/meshes/m430ia2f/collision/link_4.stl" />
+					<mesh filename="package://fanuc_config/meshes/m430ia2f/collision/link_4.stl"/>
 				</geometry>
 			</collision>
@@ -90,88 +90,63 @@
 		<link name="${prefix}link_5">
 			<visual>
-				<origin xyz="0 0 0" rpy="0 0 0" />
+				<origin xyz="0 0 0" rpy="0 0 0"/>
 				<geometry>
-					<mesh filename="package://fanuc_config/meshes/m430ia2f/visual/link_5.stl" />
+					<mesh filename="package://fanuc_config/meshes/m430ia2f/visual/link_5.stl"/>
 				</geometry>
 				<material name="">
-					<color rgba="0.75294 0.75294 0.75294 1" />
+					<color rgba="0.75294 0.75294 0.75294 1"/>
 				</material>
 			</visual>
 			<collision>
-				<origin xyz="0 0 0" rpy="0 0 0" />
+				<origin xyz="0 0 0" rpy="0 0 0"/>
 				<geometry>
-					<mesh filename="package://fanuc_config/meshes/m430ia2f/collision/link_5.stl" />
+					<mesh filename="package://fanuc_config/meshes/m430ia2f/collision/link_5.stl"/>
 				</geometry>
 			</collision>
 		</link>
-        <link name="${prefix}tool0"/>
-        <!-- joints -->
-        <joint name="${prefix}joint_1" type="revolute">
-            <origin xyz="-6.0758E-19 1.2493E-16 0.44" rpy="0 0 0" />
-            <parent link="${prefix}base_link" />
-            <child link="${prefix}link_1" />
-            <axis xyz="0 0 1" />
-            <limit lower="-3.1415" upper="3.1415" effort="0"
-                velocity="5.23598775598" />
-            <!-- calibration rising="0" falling="0" />
-            <dynamics damping="0" friction="0" />
-            <safety_controller soft_lower_limit="0"
-                soft_upper_limit="0" k_position="0" k_velocity="0" / -->
-        </joint>
-        <joint name="${prefix}joint_2" type="revolute">
-            <origin xyz="-1.4097E-17 0.171 -4.4409E-16" rpy="0 0 0" />
-            <parent link="${prefix}link_1" />
-            <child link="${prefix}link_2" />
-            <axis xyz="0 1 0" />
-            <limit lower="-2.00707" upper="2.00707" effort="0"
-                velocity="5.58505360638" />
-            <!-- calibration rising="0" falling="0" />
-            <dynamics damping="0" friction="0" />
-            <safety_controller soft_lower_limit="0"
-                soft_upper_limit="0" k_position="0" k_velocity="0" / -->
-        </joint>
-        <joint name="${prefix}joint_3" type="revolute">
-            <!-- origin xyz="1.2197E-19 -0.171 0.403" rpy="0 0 0" / -->
-            <origin xyz="1.2197E-19 -0.171 0.350" rpy="0 0 0" />
-            <parent link="${prefix}link_2" />
-            <child link="${prefix}link_3" />
-            <axis xyz="0 1 0" />
-            <limit lower="-1.771457" upper="1.771457" effort="0"
-                velocity="5.58505360638" />
-            <!-- calibration rising="0" falling="0" />
-            <dynamics damping="0" friction="0" />
-            <safety_controller soft_lower_limit="0"
-                soft_upper_limit="0" k_position="0" k_velocity="0" / -->
-        </joint>
-        <joint name="${prefix}joint_4" type="revolute">
-            <!-- origin xyz="-2.6075E-17 -0.06 0.497" rpy="0 0 0" / -->
-            <origin xyz="-2.6075E-17 -0.06 0.55" rpy="0 0 0" />
-            <parent link="${prefix}link_3" />
-            <child link="${prefix}link_4" />
-            <axis xyz="0 1 0" />
-            <limit lower="-2.617917" upper="2.617917" effort="0"
-                velocity="6.28318530718" />
-            <!-- calibration rising="0" falling="0" />
-            <dynamics damping="0" friction="0" />
-            <safety_controller soft_lower_limit="0"
-                soft_upper_limit="0" k_position="0" k_velocity="0" / -->
-        </joint>
+		<link name="${prefix}tool0"/>
+		<!-- joints -->
+		<joint name="${prefix}joint_1" type="revolute">
+			<origin xyz="-6.0758E-19 1.2493E-16 0.44" rpy="0 0 0"/>
+			<parent link="${prefix}base_link"/>
+			<child link="${prefix}link_1"/>
+			<axis xyz="0 0 1"/>
+			<limit lower="-3.1415" upper="3.1415" effort="0" velocity="5.23598775598"/>
+		</joint>
+		<joint name="${prefix}joint_2" type="revolute">
+			<origin xyz="-1.4097E-17 0.171 -4.4409E-16" rpy="0 0 0"/>
+			<parent link="${prefix}link_1"/>
+			<child link="${prefix}link_2"/>
+			<axis xyz="0 1 0"/>
+			<limit lower="-2.00707" upper="2.00707" effort="0" velocity="5.58505360638"/>
+		</joint>
+		<joint name="${prefix}joint_3" type="revolute">
+			<!-- origin xyz="1.2197E-19 -0.171 0.403" rpy="0 0 0" / -->
+			<origin xyz="1.2197E-19 -0.171 0.350" rpy="0 0 0"/>
+			<parent link="${prefix}link_2"/>
+			<child link="${prefix}link_3"/>
+			<axis xyz="0 1 0"/>
+			<limit lower="-1.771457" upper="1.771457" effort="0" velocity="5.58505360638"/>
+		</joint>
+		<joint name="${prefix}joint_4" type="revolute">
+			<!-- origin xyz="-2.6075E-17 -0.06 0.497" rpy="0 0 0" / -->
+			<origin xyz="-2.6075E-17 -0.06 0.55" rpy="0 0 0"/>
+			<parent link="${prefix}link_3"/>
+			<child link="${prefix}link_4"/>
+			<axis xyz="0 1 0"/>
+			<limit lower="-2.617917" upper="2.617917" effort="0" velocity="6.28318530718"/>
+		</joint>
 		<joint name="${prefix}joint_5" type="revolute">
-			<origin xyz="1.4734E-16 -0.035 0.065" rpy="0 0 0" />
-			<parent link="${prefix}link_4" />
-			<child link="${prefix}link_5" />
-			<axis xyz="0 0 1" />
-			<limit lower="-4.71225" upper="4.71225" effort="0"
-                velocity="20.9439510239" />
-            <!-- calibration rising="0" falling="0" />
-            <dynamics damping="0" friction="0" />
-            <safety_controller soft_lower_limit="0"
-                soft_upper_limit="0" k_position="0" k_velocity="0" / -->
+			<origin xyz="1.4734E-16 -0.035 0.065" rpy="0 0 0"/>
+			<parent link="${prefix}link_4"/>
+			<child link="${prefix}link_5"/>
+			<axis xyz="0 0 1"/>
+			<limit lower="-4.71225" upper="4.71225" effort="0" velocity="20.9439510239"/>
 		</joint>
-        <joint name="${prefix}joint_5-tool0" type="fixed">
-            <parent link="${prefix}link_5"/>
-            <child link="${prefix}tool0"/>
-            <origin xyz="0 0 0" rpy="0 0 0"/>
-        </joint>
-    </xacro:macro>
+		<joint name="${prefix}joint_5-tool0" type="fixed">
+			<parent link="${prefix}link_5"/>
+			<child link="${prefix}tool0"/>
+			<origin xyz="0 0 0" rpy="0 0 0"/>
+		</joint>
+	</xacro:macro>
 </robot>

Commit message: Add missing 'prefix' substitutions in joint declaration blocks for M-10iA and M-16iB20.

File: fanuc_config/urdf/m10ia_macro.xacro (robot description, xacro)
@@ -118,6 +118,6 @@
 		<joint name="${prefix}joint_1" type="revolute">
 			<origin xyz="0 0 0" rpy="0 0 0"/>
-			<parent link="base_link"/>
-			<child link="link_1"/>
+			<parent link="${prefix}base_link"/>
+			<child link="${prefix}link_1"/>
 			<axis xyz="0 0 1"/>
 			<limit lower="-3.14" upper="3.14" effort="0" velocity="3.67"/>
@@ -125,6 +125,6 @@
 		<joint name="${prefix}joint_2" type="revolute">
 			<origin xyz="0.15 -0.04 0.45" rpy="0 0 0"/>
-			<parent link="link_1"/>
-			<child link="link_2"/>
+			<parent link="${prefix}link_1"/>
+			<child link="${prefix}link_2"/>
 			<axis xyz="0 1 0"/>
 			<limit lower="-1.57" upper="2.79" effort="0" velocity="3.32"/>
@@ -132,6 +132,6 @@
 		<joint name="${prefix}joint_3" type="revolute">
 			<origin xyz="0 -0.0225 0.6" rpy="0 0 0"/>
-			<parent link="link_2"/>
-			<child link="link_3"/>
+			<parent link="${prefix}link_2"/>
+			<child link="${prefix}link_3"/>
 			<axis xyz="0 -1 0"/>
 			<limit lower="-3.14" upper="4.61" effort="0" velocity="3.67"/>
@@ -139,6 +139,6 @@
 		<joint name="${prefix}joint_4" type="revolute">
 			<origin xyz="0.1805 0.0625 0.2" rpy="0 0 0"/>
-			<parent link="link_3"/>
-			<child link="link_4"/>
+			<parent link="${prefix}link_3"/>
+			<child link="${prefix}link_4"/>
 			<axis xyz="-1 0 0"/>
 			<limit lower="-3.31" upper="3.31" effort="0" velocity="6.98"/>
@@ -146,6 +146,6 @@
 		<joint name="${prefix}joint_5" type="revolute">
 			<origin xyz="0.4595 -0.0565 0" rpy="0 0 0"/>
-			<parent link="link_4"/>
-			<child link="link_5"/>
+			<parent link="${prefix}link_4"/>
+			<child link="${prefix}link_5"/>
 			<axis xyz="0 -1 0"/>
 			<limit lower="-3.31" upper="3.31" effort="0" velocity="6.98"/>
@@ -153,12 +153,12 @@
 		<joint name="${prefix}joint_6" type="revolute">
 			<origin xyz="0.1 0.0565 0" rpy="0 0 0"/>
-			<parent link="link_5"/>
-			<child link="link_6"/>
+			<parent link="${prefix}link_5"/>
+			<child link="${prefix}link_6"/>
 			<axis xyz="-1 0 0"/>
 			<limit lower="-6.28" upper="6.28" effort="0" velocity="10.47"/>
 		</joint>
 		<joint name="${prefix}joint_6-tool0" type="fixed">
-			<parent link="link_6"/>
-			<child link="tool0"/>
+			<parent link="${prefix}link_6"/>
+			<child link="${prefix}tool0"/>
 			<origin xyz="0.1 0.0565 0" rpy="0 0 0"/>
 		</joint>

File: fanuc_config/urdf/m16ib20_macro.xacro (robot description, xacro)
@@ -116,6 +116,6 @@
 		<joint name="${prefix}joint_1" type="revolute">
 			<origin xyz="0 0 0.245" rpy="0 0 0"/>
-			<parent link="base_link"/>
-			<child link="link_1"/>
+			<parent link="${prefix}base_link"/>
+			<child link="${prefix}link_1"/>
 			<axis xyz="0 0 1"/>
 			<limit lower="-2.967" upper="2.967" effort="0" velocity="2.879"/>
@@ -123,6 +123,6 @@
 		<joint name="${prefix}joint_2" type="revolute">
 			<origin xyz="0.15 0.18759 0.28" rpy="0 0 0"/>
-			<parent link="link_1"/>
-			<child link="link_2"/>
+			<parent link="${prefix}link_1"/>
+			<child link="${prefix}link_2"/>
 			<axis xyz="0 1 0"/>
 			<limit lower="-1.38" upper="2.78" effort="0" velocity="2.879"/>
@@ -130,6 +130,6 @@
 		<joint name="${prefix}joint_3" type="revolute">
 			<origin xyz="0 -0.18759 0.77" rpy="0 0 0"/>
-			<parent link="link_2"/>
-			<child link="link_3"/>
+			<parent link="${prefix}link_2"/>
+			<child link="${prefix}link_3"/>
 			<axis xyz="0 -1 0"/>
 			<limit lower="-4.08" upper="1.38" effort="0" velocity="3.054"/>
@@ -137,6 +137,6 @@
 		<joint name="${prefix}joint_4" type="revolute">
 			<origin xyz="0.18425 0 0.1" rpy="0 0 0"/>
-			<parent link="link_3"/>
-			<child link="link_4"/>
+			<parent link="${prefix}link_3"/>
+			<child link="${prefix}link_4"/>
 			<axis xyz="-1 0 0"/>
 			<limit lower="-3.48" upper="3.48" effort="0" velocity="6.108"/>
@@ -144,6 +144,6 @@
 		<joint name="${prefix}joint_5" type="revolute">
 			<origin xyz="0.55575 0 0" rpy="0 0 0"/>
-			<parent link="link_4"/>
-			<child link="link_5"/>
+			<parent link="${prefix}link_4"/>
+			<child link="${prefix}link_5"/>
 			<axis xyz="0 -1 0"/>
 			<limit lower="-2.43" upper="2.43" effort="0" velocity="5.934"/>
@@ -151,6 +151,6 @@
 		<joint name="${prefix}joint_6" type="revolute">
 			<origin xyz="0.1 0 0" rpy="0 0 0"/>
-			<parent link="link_5"/>
-			<child link="link_6"/>
+			<parent link="${prefix}link_5"/>
+			<child link="${prefix}link_6"/>
 			<axis xyz="-1 0 0"/>
 			<limit lower="-7.84" upper="7.84" effort="0" velocity="9.075"/>
