Commit message: Make naming more consistent across launch files, URDFs and directories.
Arm navigation packages will be fixed as well.

File: fanuc_config/urdf/m10ia.urdf (robot description, URDF)
Before this commit: robot m10iA, 8 links, 7 joints
Links:
- link base_link: geometry collision mesh filename=package://fanuc_config/meshes/m10ia/collision/base_link.stl; visual mesh filename=package://fanuc_config/meshes/m10ia/visual/base_link.stl
- link link_1: geometry collision mesh filename=package://fanuc_config/meshes/m10ia/collision/link_1.stl; visual mesh filename=package://fanuc_config/meshes/m10ia/visual/link_1.stl
- link link_2: geometry collision mesh filename=package://fanuc_config/meshes/m10ia/collision/link_2.stl; visual mesh filename=package://fanuc_config/meshes/m10ia/visual/link_2.stl
- link link_3: geometry collision mesh filename=package://fanuc_config/meshes/m10ia/collision/link_3.stl; visual mesh filename=package://fanuc_config/meshes/m10ia/visual/link_3.stl
- link link_4: geometry collision mesh filename=package://fanuc_config/meshes/m10ia/collision/link_4.stl; visual mesh filename=package://fanuc_config/meshes/m10ia/visual/link_4.stl
- link link_5: geometry collision mesh filename=package://fanuc_config/meshes/m10ia/collision/link_5.stl; visual mesh filename=package://fanuc_config/meshes/m10ia/visual/link_5.stl
- link link_6: geometry collision mesh filename=package://fanuc_config/meshes/m10ia/collision/link_6.stl; visual mesh filename=package://fanuc_config/meshes/m10ia/visual/link_6.stl

File: fanuc_config/urdf/m10ia_macro.xacro (robot description, xacro)
@@ -1,5 +1,5 @@
 <?xml version="1.0" ?>
 <robot xmlns:xacro="http://ros.org/wiki/xacro">
-	<xacro:macro name="m10iA" params="prefix">
+	<xacro:macro name="m10ia" params="prefix">
 		<!-- link list -->
 		<link name="${prefix}base_link">
@@ -10,5 +10,5 @@
       			<geometry>
         			<mesh
-          			filename="package://fanuc_config/meshes/m_10iA/visual/base_link.stl" />
+          			filename="package://fanuc_config/meshes/m10ia/visual/base_link.stl" />
       			</geometry>
       			<material
@@ -23,5 +23,5 @@
        			rpy="-1.578 0 0" />
 				<geometry>
-					<mesh filename="package://fanuc_config/meshes/m_10iA/collision/base_link.stl" />
+					<mesh filename="package://fanuc_config/meshes/m10ia/collision/base_link.stl" />
 				</geometry>
 				<material name="yellow">
@@ -37,5 +37,5 @@
       			<geometry>
         			<mesh
-          			filename="package://fanuc_config/meshes/m_10iA/visual/link_1.stl" />
+          			filename="package://fanuc_config/meshes/m10ia/visual/link_1.stl" />
       			</geometry>
       			<material name="grey"/>
@@ -46,5 +46,5 @@
         			rpy="0 0 0" />
 				<geometry>
-					<mesh filename="package://fanuc_config/meshes/m_10iA/collision/link_1.stl" />
+					<mesh filename="package://fanuc_config/meshes/m10ia/collision/link_1.stl" />
 				</geometry>
 				<material name="yellow"/>
@@ -58,5 +58,5 @@
       			<geometry>
         			<mesh
-          			filename="package://fanuc_config/meshes/m_10iA/visual/link_2.stl" />
+          			filename="package://fanuc_config/meshes/m10ia/visual/link_2.stl" />
       			</geometry>
       			<material name="grey"/>
@@ -67,5 +67,5 @@
         			rpy="0 0 0" />
 				<geometry>
-					<mesh filename="package://fanuc_config/meshes/m_10iA/collision/link_2.stl" />
+					<mesh filename="package://fanuc_config/meshes/m10ia/collision/link_2.stl" />
 				</geometry>
 				<material name="yellow"/>
@@ -79,5 +79,5 @@
 			  	<geometry>
 					<mesh
-				  	filename="package://fanuc_config/meshes/m_10iA/visual/link_3.stl" />
+				  	filename="package://fanuc_config/meshes/m10ia/visual/link_3.stl" />
 			  	</geometry>
 			  	<material name="grey"/>
@@ -88,5 +88,5 @@
         			rpy="0 0 0" />
 				<geometry>
-					<mesh filename="package://fanuc_config/meshes/m_10iA/collision/link_3.stl" />
+					<mesh filename="package://fanuc_config/meshes/m10ia/collision/link_3.stl" />
 				</geometry>
 				<material name="yellow"/>
@@ -100,5 +100,5 @@
 				  <geometry>
 					<mesh
-					  filename="package://fanuc_config/meshes/m_10iA/visual/link_4.stl" />
+					  filename="package://fanuc_config/meshes/m10ia/visual/link_4.stl" />
 				  </geometry>
 				  <material name="grey"/>
@@ -109,5 +109,5 @@
         			rpy="0 0 0" />
 				<geometry>
-					<mesh filename="package://fanuc_config/meshes/m_10iA/collision/link_4.stl" />
+					<mesh filename="package://fanuc_config/meshes/m10ia/collision/link_4.stl" />
 				</geometry>
 				<material name="yellow"/>
@@ -121,5 +121,5 @@
 				<geometry>
 					<mesh
-					  filename="package://fanuc_config/meshes/m_10iA/visual/link_5.stl" />
+					  filename="package://fanuc_config/meshes/m10ia/visual/link_5.stl" />
 				</geometry>
 				<material name="grey"/>
@@ -130,5 +130,5 @@
         			rpy="0 0 0" />
 				<geometry>
-					<mesh filename="package://fanuc_config/meshes/m_10iA/collision/link_5.stl" />
+					<mesh filename="package://fanuc_config/meshes/m10ia/collision/link_5.stl" />
 				</geometry>
 				<material name="yellow"/>
@@ -142,5 +142,5 @@
 				<geometry>
 					<mesh
-					  filename="package://fanuc_config/meshes/m_10iA/visual/link_6.stl" />
+					  filename="package://fanuc_config/meshes/m10ia/visual/link_6.stl" />
 				</geometry>
 				<material name="grey"/>
@@ -151,5 +151,5 @@
         			rpy="0 0 0" />
 				<geometry>
-					<mesh filename="package://fanuc_config/meshes/m_10iA/collision/link_6.stl" />
+					<mesh filename="package://fanuc_config/meshes/m10ia/collision/link_6.stl" />
 				</geometry>
 				<material name="yellow"/>

File: fanuc_config/urdf/m16ib20.urdf (robot description, URDF)
Before this commit: robot M16iB20, 8 links, 7 joints
Links:
- link base_link: geometry collision mesh filename=package://fanuc_config/meshes/m16ib20/collision/base_link.S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; visual mesh filename=package://fanuc_config/meshes/m16ib20/visual/base_link.STL
- link link_1: geometry collision mesh filename=package://fanuc_config/meshes/m16ib20/collision/Link_1.STL; visual mesh filename=package://fanuc_config/meshes/m16ib20/visual/Link_1.STL
- link link_2: geometry collision mesh filename=package://fanuc_config/meshes/m16ib20/collision/Link_2.STL; visual mesh filename=package://fanuc_config/meshes/m16ib20/visual/Link_2.STL
- link link_3: geometry collision mesh filename=package://fanuc_config/meshes/m16ib20/collision/Link_3.STL; visual mesh filename=package://fanuc_config/meshes/m16ib20/visual/Link_3.STL
- link link_4: geometry collision mesh filename=package://fanuc_config/meshes/m16ib20/collision/Link_4.STL; visual mesh filename=package://fanuc_config/meshes/m16ib20/visual/Link_4.STL
- link link_5: geometry collision mesh filename=package://fanuc_config/meshes/m16ib20/collision/Link_5.STL; visual mesh filename=package://fanuc_config/meshes/m16ib20/visual/Link_5.STL
- link link_6: geometry collision mesh filename=package://fanuc_config/meshes/m16ib20/collision/Link_6.STL; visual mesh filename=package://fanuc_config/meshes/m16ib20/visual/Link_6.STL

File: fanuc_config/urdf/m16ib20_macro.xacro (robot description, xacro)
@@ -1,5 +1,5 @@
 <?xml version="1.0" ?>
 <robot xmlns:xacro="http://ros.org/wiki/xacro">
-	<xacro:macro name="M16iB20" params="prefix">
+	<xacro:macro name="m16ib20" params="prefix">
 	<!-- links -->
 		  <link name="${prefix}base_link">
@@ -10,19 +10,19 @@
 		      <geometry>
 			<mesh
-			  filename="package://fanuc_config/meshes/m_16iB20/visual/base_link.STL" />
-		      </geometry>
-		      <material
-			name="">
-			<color
-			  rgba="1 1 0 1" />
-		      </material>
-		    </visual>
-		    <collision>
-		      <origin
-			xyz="0 0 0"
-			rpy="0 0 0" />
-		      <geometry>
-			<mesh
-			  filename="package://fanuc_config/meshes/m_16iB20/collision/base_link.STL" />
+			  filename="package://fanuc_config/meshes/m16ib20/visual/base_link.STL" />
+		      </geometry>
+		      <material
+			name="">
+			<color
+			  rgba="1 1 0 1" />
+		      </material>
+		    </visual>
+		    <collision>
+		      <origin
+			xyz="0 0 0"
+			rpy="0 0 0" />
+		      <geometry>
+			<mesh
+			  filename="package://fanuc_config/meshes/m16ib20/collision/base_link.STL" />
 		      </geometry>
 		    </collision>
@@ -35,19 +35,19 @@
 		      <geometry>
 			<mesh
-			  filename="package://fanuc_config/meshes/m_16iB20/visual/Link_1.STL" />
-		      </geometry>
-		      <material
-			name="">
-			<color
-			  rgba="1 1 0 1" />
-		      </material>
-		    </visual>
-		    <collision>
-		      <origin
-			xyz="0 0 0"
-			rpy="0 0 0" />
-		      <geometry>
-			<mesh
-			  filename="package://fanuc_config/meshes/m_16iB20/collision/Link_1.STL" />
+			  filename="package://fanuc_config/meshes/m16ib20/visual/Link_1.STL" />
+		      </geometry>
+		      <material
+			name="">
+			<color
+			  rgba="1 1 0 1" />
+		      </material>
+		    </visual>
+		    <collision>
+		      <origin
+			xyz="0 0 0"
+			rpy="0 0 0" />
+		      <geometry>
+			<mesh
+			  filename="package://fanuc_config/meshes/m16ib20/collision/Link_1.STL" />
 		      </geometry>
 		    </collision>
@@ -60,19 +60,19 @@
 		      <geometry>
 			<mesh
-			  filename="package://fanuc_config/meshes/m_16iB20/visual/Link_2.STL" />
-		      </geometry>
-		      <material
-			name="">
-			<color
-			  rgba="1 1 0 1" />
-		      </material>
-		    </visual>
-		    <collision>
-		      <origin
-			xyz="0 0 0"
-			rpy="0 0 0" />
-		      <geometry>
-			<mesh
-			  filename="package://fanuc_config/meshes/m_16iB20/collision/Link_2.STL" />
+			  filename="package://fanuc_config/meshes/m16ib20/visual/Link_2.STL" />
+		      </geometry>
+		      <material
+			name="">
+			<color
+			  rgba="1 1 0 1" />
+		      </material>
+		    </visual>
+		    <collision>
+		      <origin
+			xyz="0 0 0"
+			rpy="0 0 0" />
+		      <geometry>
+			<mesh
+			  filename="package://fanuc_config/meshes/m16ib20/collision/Link_2.STL" />
 		      </geometry>
 		    </collision>
@@ -85,19 +85,19 @@
 		      <geometry>
 			<mesh
-			  filename="package://fanuc_config/meshes/m_16iB20/visual/Link_3.STL" />
-		      </geometry>
-		      <material
-			name="">
-			<color
-			  rgba="1 1 0 1" />
-		      </material>
-		    </visual>
-		    <collision>
-		      <origin
-			xyz="0 0 0"
-			rpy="0 0 0" />
-		      <geometry>
-			<mesh
-			  filename="package://fanuc_config/meshes/m_16iB20/collision/Link_3.STL" />
+			  filename="package://fanuc_config/meshes/m16ib20/visual/Link_3.STL" />
+		      </geometry>
+		      <material
+			name="">
+			<color
+			  rgba="1 1 0 1" />
+		      </material>
+		    </visual>
+		    <collision>
+		      <origin
+			xyz="0 0 0"
+			rpy="0 0 0" />
+		      <geometry>
+			<mesh
+			  filename="package://fanuc_config/meshes/m16ib20/collision/Link_3.STL" />
 		      </geometry>
 		    </collision>
@@ -110,19 +110,19 @@
 		      <geometry>
 			<mesh
-			  filename="package://fanuc_config/meshes/m_16iB20/visual/Link_4.STL" />
-		      </geometry>
-		      <material
-			name="">
-			<color
-			  rgba="1 1 0 1" />
-		      </material>
-		    </visual>
-		    <collision>
-		      <origin
-			xyz="0 0 0"
-			rpy="0 0 0" />
-		      <geometry>
-			<mesh
-			  filename="package://fanuc_config/meshes/m_16iB20/collision/Link_4.STL" />
+			  filename="package://fanuc_config/meshes/m16ib20/visual/Link_4.STL" />
+		      </geometry>
+		      <material
+			name="">
+			<color
+			  rgba="1 1 0 1" />
+		      </material>
+		    </visual>
+		    <collision>
+		      <origin
+			xyz="0 0 0"
+			rpy="0 0 0" />
+		      <geometry>
+			<mesh
+			  filename="package://fanuc_config/meshes/m16ib20/collision/Link_4.STL" />
 		      </geometry>
 		    </collision>
@@ -135,19 +135,19 @@
 		      <geometry>
 			<mesh
-			  filename="package://fanuc_config/meshes/m_16iB20/visual/Link_5.STL" />
-		      </geometry>
-		      <material
-			name="">
-			<color
-			  rgba="1 1 0 1" />
-		      </material>
-		    </visual>
-		    <collision>
-		      <origin
-			xyz="0 0 0"
-			rpy="0 0 0" />
-		      <geometry>
-			<mesh
-			  filename="package://fanuc_config/meshes/m_16iB20/collision/Link_5.STL" />
+			  filename="package://fanuc_config/meshes/m16ib20/visual/Link_5.STL" />
+		      </geometry>
+		      <material
+			name="">
+			<color
+			  rgba="1 1 0 1" />
+		      </material>
+		    </visual>
+		    <collision>
+		      <origin
+			xyz="0 0 0"
+			rpy="0 0 0" />
+		      <geometry>
+			<mesh
+			  filename="package://fanuc_config/meshes/m16ib20/collision/Link_5.STL" />
 		      </geometry>
 		    </collision>
@@ -160,19 +160,19 @@
 		      <geometry>
 			<mesh
-			  filename="package://fanuc_config/meshes/m_16iB20/visual/Link_6.STL" />
-		      </geometry>
-		      <material
-			name="">
-			<color
-			  rgba="1 1 0 1" />
-		      </material>
-		    </visual>
-		    <collision>
-		      <origin
-			xyz="0 0 0"
-			rpy="0 0 0" />
-		      <geometry>
-			<mesh
-			  filename="package://fanuc_config/meshes/m_16iB20/collision/Link_6.STL" />
+			  filename="package://fanuc_config/meshes/m16ib20/visual/Link_6.STL" />
+		      </geometry>
+		      <material
+			name="">
+			<color
+			  rgba="1 1 0 1" />
+		      </material>
+		    </visual>
+		    <collision>
+		      <origin
+			xyz="0 0 0"
+			rpy="0 0 0" />
+		      <geometry>
+			<mesh
+			  filename="package://fanuc_config/meshes/m16ib20/collision/Link_6.STL" />
 		      </geometry>
 		    </collision>

File: fanuc_config/urdf/m430ia2f.urdf (robot description, URDF)
Before this commit: robot m430iA2F, 7 links, 6 joints
Links:
- link base_link: geometry collision mesh filename=package://fanuc_config/meshes/m430ia2f/collision/base_link.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; visual mesh filename=package://fanuc_config/meshes/m430ia2f/visual/base_link.stl
- link link_1: geometry collision mesh filename=package://fanuc_config/meshes/m430ia2f/collision/link_1.stl; visual mesh filename=package://fanuc_config/meshes/m430ia2f/visual/link_1.stl
- link link_2: geometry collision mesh filename=package://fanuc_config/meshes/m430ia2f/collision/link_2.stl; visual mesh filename=package://fanuc_config/meshes/m430ia2f/visual/link_2.stl
- link link_3: geometry collision mesh filename=package://fanuc_config/meshes/m430ia2f/collision/link_3.stl; visual mesh filename=package://fanuc_config/meshes/m430ia2f/visual/link_3.stl
- link link_4: geometry collision mesh filename=package://fanuc_config/meshes/m430ia2f/collision/link_4.stl; visual mesh filename=package://fanuc_config/meshes/m430ia2f/visual/link_4.stl
- link link_5: geometry collision mesh filename=package://fanuc_config/meshes/m430ia2f/collision/link_5.stl; visual mesh filename=package://fanuc_config/meshes/m430ia2f/visual/link_5.stl

File: fanuc_config/urdf/m430ia2f_macro.xacro (robot description, xacro)
@@ -1,5 +1,5 @@
 <?xml version="1.0" ?>
 <robot xmlns:xacro="http://ros.org/wiki/xacro">
-    <xacro:macro name="m430iA2F" params="prefix">
+    <xacro:macro name="m430ia2f" params="prefix">
         <!-- links -->
 		<link name="${prefix}base_link">
@@ -7,5 +7,5 @@
 				<origin xyz="0 0 0" rpy="0 0 0" />
 				<geometry>
-					<mesh filename="package://fanuc_config/meshes/m_430iA/visual/base_link.stl" />
+					<mesh filename="package://fanuc_config/meshes/m430ia2f/visual/base_link.stl" />
 				</geometry>
 				<material name="white">
@@ -16,5 +16,5 @@
 				<origin xyz="0 0 0" rpy="0 0 0" />
 				<geometry>
-					<mesh filename="package://fanuc_config/meshes/m_430iA/collision/base_link.stl" />
+					<mesh filename="package://fanuc_config/meshes/m430ia2f/collision/base_link.stl" />
 				</geometry>
 			</collision>
@@ -24,5 +24,5 @@
 				<origin xyz="0 0 0" rpy="0 0 0" />
 				<geometry>
-					<mesh filename="package://fanuc_config/meshes/m_430iA/visual/link_1.stl" />
+					<mesh filename="package://fanuc_config/meshes/m430ia2f/visual/link_1.stl" />
 				</geometry>
 				<material name="">
@@ -33,5 +33,5 @@
 				<origin xyz="0 0 0" rpy="0 0 0" />
 				<geometry>
-					<mesh filename="package://fanuc_config/meshes/m_430iA/collision/link_1.stl" />
+					<mesh filename="package://fanuc_config/meshes/m430ia2f/collision/link_1.stl" />
 				</geometry>
 			</collision>
@@ -41,5 +41,5 @@
 				<origin xyz="0 0 0" rpy="0 0 0" />
 				<geometry>
-					<mesh filename="package://fanuc_config/meshes/m_430iA/visual/link_2.stl" />
+					<mesh filename="package://fanuc_config/meshes/m430ia2f/visual/link_2.stl" />
 				</geometry>
 				<material name="">
@@ -50,5 +50,5 @@
 				<origin xyz="0 0 0" rpy="0 0 0" />
 				<geometry>
-					<mesh filename="package://fanuc_config/meshes/m_430iA/collision/link_2.stl" />
+					<mesh filename="package://fanuc_config/meshes/m430ia2f/collision/link_2.stl" />
 				</geometry>
 			</collision>
@@ -58,5 +58,5 @@
 				<origin xyz="0 0 0.053" rpy="0 0 0" />
 				<geometry>
-					<mesh filename="package://fanuc_config/meshes/m_430iA/visual/link_3.stl" />
+					<mesh filename="package://fanuc_config/meshes/m430ia2f/visual/link_3.stl" />
 				</geometry>
 				<material name="">
@@ -67,5 +67,5 @@
 				<origin xyz="0 0 0.053" rpy="0 0 0" />
 				<geometry>
-					<mesh filename="package://fanuc_config/meshes/m_430iA/collision/link_3.stl" />
+					<mesh filename="package://fanuc_config/meshes/m430ia2f/collision/link_3.stl" />
 				</geometry>
 			</collision>
@@ -75,5 +75,5 @@
 				<origin xyz="0 0 0" rpy="0 0 0" />
 				<geometry>
-					<mesh filename="package://fanuc_config/meshes/m_430iA/visual/link_4.stl" />
+					<mesh filename="package://fanuc_config/meshes/m430ia2f/visual/link_4.stl" />
 				</geometry>
 				<material name="">
@@ -84,5 +84,5 @@
 				<origin xyz="0 0 0" rpy="0 0 0" />
 				<geometry>
-					<mesh filename="package://fanuc_config/meshes/m_430iA/collision/link_4.stl" />
+					<mesh filename="package://fanuc_config/meshes/m430ia2f/collision/link_4.stl" />
 				</geometry>
 			</collision>
@@ -92,5 +92,5 @@
 				<origin xyz="0 0 0" rpy="0 0 0" />
 				<geometry>
-					<mesh filename="package://fanuc_config/meshes/m_430iA/visual/link_5.stl" />
+					<mesh filename="package://fanuc_config/meshes/m430ia2f/visual/link_5.stl" />
 				</geometry>
 				<material name="">
@@ -101,5 +101,5 @@
 				<origin xyz="0 0 0" rpy="0 0 0" />
 				<geometry>
-					<mesh filename="package://fanuc_config/meshes/m_430iA/collision/link_5.stl" />
+					<mesh filename="package://fanuc_config/meshes/m430ia2f/collision/link_5.stl" />
 				</geometry>
 			</collision>

Commit message: Correct joint limits, velocities and directions for M-10iA. Data taken from "FANUC Robot M-10iA Mechanical Unit Operator's Manual, B-82754EN/09, page 11".

File: fanuc_config/urdf/m10ia.urdf (robot description, URDF)
Before this commit: robot m10ia, 8 links, 7 joints
Joints:
- joint joint_1: limit lower=-5.93 upper=5.93 effort=0 velocity=3.665 -> lower=-3.14 upper=3.14 effort=0 velocity=3.67
- joint joint_2: limit lower=-4.36 upper=4.36 effort=0 velocity=3.32 -> lower=-1.57 upper=2.79 effort=0 velocity=3.32
- joint joint_3: axis 0 1 0 -> 0 -1 0; limit lower=-5.06 upper=5.06 effort=0 velocity=3.665 -> lower=-3.14 upper=4.61 effort=0 velocity=3.67
- joint joint_4: axis 1 0 0 -> -1 0 0; limit lower=-6.63 upper=6.63 effort=0 velocity=6.98 -> lower=-3.31 upper=3.31 effort=0 velocity=6.98
- joint joint_5: axis 0 1 0 -> 0 -1 0; limit lower=-6.63 upper=6.63 effort=0 velocity=3.98 -> lower=-3.31 upper=3.31 effort=0 velocity=6.98
- joint joint_6: axis 1 0 0 -> -1 0 0; limit lower=-12.566 upper=12.566 effort=0 velocity=10.47 -> lower=-6.28 upper=6.28 effort=0 velocity=10.47

File: fanuc_config/urdf/m10ia_macro.xacro (robot description, xacro)
@@ -121,5 +121,5 @@
 			<child link="link_1"/>
 			<axis xyz="0 0 1"/>
-			<limit lower="-5.93" upper="5.93" effort="0" velocity="3.665"/>
+			<limit lower="-3.14" upper="3.14" effort="0" velocity="3.67"/>
 		</joint>
 		<joint name="${prefix}joint_2" type="revolute">
@@ -128,5 +128,5 @@
 			<child link="link_2"/>
 			<axis xyz="0 1 0"/>
-			<limit lower="-4.36" upper="4.36" effort="0" velocity="3.32"/>
+			<limit lower="-1.57" upper="2.79" effort="0" velocity="3.32"/>
 		</joint>
 		<joint name="${prefix}joint_3" type="revolute">
@@ -134,6 +134,6 @@
 			<parent link="link_2"/>
 			<child link="link_3"/>
-			<axis xyz="0 1 0"/>
-			<limit lower="-5.06" upper="5.06" effort="0" velocity="3.665"/>
+			<axis xyz="0 -1 0"/>
+			<limit lower="-3.14" upper="4.61" effort="0" velocity="3.67"/>
 		</joint>
 		<joint name="${prefix}joint_4" type="revolute">
@@ -141,6 +141,6 @@
 			<parent link="link_3"/>
 			<child link="link_4"/>
-			<axis xyz="1 0 0"/>
-			<limit lower="-6.63" upper="6.63" effort="0" velocity="6.98"/>
+			<axis xyz="-1 0 0"/>
+			<limit lower="-3.31" upper="3.31" effort="0" velocity="6.98"/>
 		</joint>
 		<joint name="${prefix}joint_5" type="revolute">
@@ -148,6 +148,6 @@
 			<parent link="link_4"/>
 			<child link="link_5"/>
-			<axis xyz="0 1 0"/>
-			<limit lower="-6.63" upper="6.63" effort="0" velocity="3.98"/>
+			<axis xyz="0 -1 0"/>
+			<limit lower="-3.31" upper="3.31" effort="0" velocity="6.98"/>
 		</joint>
 		<joint name="${prefix}joint_6" type="revolute">
@@ -155,6 +155,6 @@
 			<parent link="link_5"/>
 			<child link="link_6"/>
-			<axis xyz="1 0 0"/>
-			<limit lower="-12.566" upper="12.566" effort="0" velocity="10.47"/>
+			<axis xyz="-1 0 0"/>
+			<limit lower="-6.28" upper="6.28" effort="0" velocity="10.47"/>
 		</joint>
 		<joint name="${prefix}joint_6-tool0" type="fixed">

Commit message: Remove the tool0 joint offset (users with actual end-effectors will have to adjust this for their specific situation anyway, so no sense in keeping the current one).

File: fanuc_config/urdf/m10ia.urdf (robot description, URDF)
Before this commit: robot m10ia, 8 links, 7 joints
Joints:
- joint joint_6-tool0: origin xyz=0.1 0.0565 0 rpy=0 0 0 -> xyz=0 0 0 rpy=0 0 0

File: fanuc_config/urdf/m10ia_macro.xacro (robot description, xacro)
@@ -161,5 +161,5 @@
 			<parent link="${prefix}link_6"/>
 			<child link="${prefix}tool0"/>
-			<origin xyz="0.1 0.0565 0" rpy="0 0 0"/>
+			<origin xyz="0 0 0" rpy="0 0 0"/>
 		</joint>
 	</xacro:macro>
