Commit message: Update M-16iB/20 joint motion ranges and maximum velocities based on documentation and data from the controller.
NB: the previous values were taken from a M-16 that had a non-default configuration. This commit brings this support package more in-line with the others (only default configurations and limits).
NB2: no changes were observed in a regenerated arm navigation package

File: fanuc_m16ib_support/urdf/m16ib20.urdf (robot description, URDF)
Before this commit: robot fanuc_m16ib20, 8 links, 7 joints
Joints:
- joint joint_1: limit lower=-2.967 upper=2.967 effort=0 velocity=2.879 -> lower=-2.9671 upper=2.9671 effort=0 velocity=2.8798
- joint joint_2: limit lower=-1.38 upper=2.78 effort=0 velocity=2.879 -> lower=-1.5708 upper=2.7925 effort=0 velocity=2.8798
- joint joint_3: limit lower=-4.08 upper=1.38 effort=0 velocity=3.054 -> lower=-2.9671 upper=5.0615 effort=0 velocity=3.0543
- joint joint_4: limit lower=-3.48 upper=3.48 effort=0 velocity=6.108 -> lower=-3.4907 upper=3.4907 effort=0 velocity=6.1087
- joint joint_5: limit lower=-2.43 upper=2.43 effort=0 velocity=5.934 -> lower=-2.4435 upper=2.4435 effort=0 velocity=5.9341
- joint joint_6: limit lower=-7.84 upper=7.84 effort=0 velocity=9.075 -> lower=-7.8540 upper=7.8540 effort=0 velocity=9.0757

File: fanuc_m16ib_support/urdf/m16ib20_macro.xacro (robot description, xacro)
@@ -116,5 +116,5 @@
 			<child link="${prefix}link_1"/>
 			<axis xyz="0 0 1"/>
-			<limit lower="-2.967" upper="2.967" effort="0" velocity="2.879"/>
+			<limit effort="0" lower="-2.9671" upper="2.9671" velocity="2.8798" />
 		</joint>
 		<joint name="${prefix}joint_2" type="revolute">
@@ -123,5 +123,5 @@
 			<child link="${prefix}link_2"/>
 			<axis xyz="0 1 0"/>
-			<limit lower="-1.38" upper="2.78" effort="0" velocity="2.879"/>
+			<limit effort="0" lower="-1.5708" upper="2.7925" velocity="2.8798" />
 		</joint>
 		<joint name="${prefix}joint_3" type="revolute">
@@ -130,5 +130,5 @@
 			<child link="${prefix}link_3"/>
 			<axis xyz="0 -1 0"/>
-			<limit lower="-4.08" upper="1.38" effort="0" velocity="3.054"/>
+			<limit effort="0" lower="-2.9671" upper="5.0615" velocity="3.0543" />
 		</joint>
 		<joint name="${prefix}joint_4" type="revolute">
@@ -137,5 +137,5 @@
 			<child link="${prefix}link_4"/>
 			<axis xyz="-1 0 0"/>
-			<limit lower="-3.48" upper="3.48" effort="0" velocity="6.108"/>
+			<limit effort="0" lower="-3.4907" upper="3.4907" velocity="6.1087" />
 		</joint>
 		<joint name="${prefix}joint_5" type="revolute">
@@ -144,5 +144,5 @@
 			<child link="${prefix}link_5"/>
 			<axis xyz="0 -1 0"/>
-			<limit lower="-2.43" upper="2.43" effort="0" velocity="5.934"/>
+			<limit effort="0" lower="-2.4435" upper="2.4435" velocity="5.9341" />
 		</joint>
 		<joint name="${prefix}joint_6" type="revolute">
@@ -151,5 +151,5 @@
 			<child link="${prefix}link_6"/>
 			<axis xyz="-1 0 0"/>
-			<limit lower="-7.84" upper="7.84" effort="0" velocity="9.075"/>
+			<limit effort="0" lower="-7.8540" upper="7.8540" velocity="9.0757" />
 		</joint>
 		<joint name="${prefix}joint_6-tool0" type="fixed">

Commit message: m16ib: update urdfs based on DH data. For #54 and #63.

File: fanuc_m16ib_support/urdf/m16ib20.urdf (robot description, URDF)
Before this commit: robot fanuc_m16ib20, 8 links, 7 joints
Joints:
- joint joint_1: origin xyz=0 0 0.245 rpy=0 0 0 -> xyz=0 0 0.525 rpy=0 0 0
- joint joint_2: origin xyz=0.15 0.18759 0.28 rpy=0 0 0 -> xyz=0.150 0 0 rpy=0 0 0
- joint joint_3: origin xyz=0 -0.18759 0.77 rpy=0 0 0 -> xyz=0 0 0.770 rpy=0 0 0
- joint joint_4: origin xyz=0.18425 0 0.1 rpy=0 0 0 -> xyz=0 0 0.100 rpy=0 0 0
- joint joint_5: origin xyz=0.55575 0 0 rpy=0 0 0 -> xyz=0.740 0 0 rpy=0 0 0
- joint joint_6: origin xyz=0.1 0 0 rpy=0 0 0 -> xyz=0.100 0 0 rpy=0 0 0
- joint joint_6-tool0: origin xyz=0 0 0 rpy=0 0 0 -> xyz=0 0 0 rpy=3.1415926535 -1.570796327 0

File: fanuc_m16ib_support/urdf/m16ib20_macro.xacro (robot description, xacro)
@@ -2,4 +2,5 @@
 <robot xmlns:xacro="http://ros.org/wiki/xacro">
 	<xacro:include filename="$(find fanuc_resources)/urdf/common_materials.xacro"/>
+	<xacro:include filename="$(find fanuc_resources)/urdf/common_constants.xacro"/>
 	<xacro:macro name="fanuc_m16ib20" params="prefix">
 		<!-- links -->
@@ -112,5 +113,5 @@
 		<!-- joints -->
 		<joint name="${prefix}joint_1" type="revolute">
-			<origin xyz="0 0 0.245" rpy="0 0 0"/>
+			<origin xyz="0 0 0.525" rpy="0 0 0"/>
 			<parent link="${prefix}base_link"/>
 			<child link="${prefix}link_1"/>
@@ -119,5 +120,5 @@
 		</joint>
 		<joint name="${prefix}joint_2" type="revolute">
-			<origin xyz="0.15 0.18759 0.28" rpy="0 0 0"/>
+			<origin xyz="0.150 0 0" rpy="0 0 0"/>
 			<parent link="${prefix}link_1"/>
 			<child link="${prefix}link_2"/>
@@ -126,5 +127,5 @@
 		</joint>
 		<joint name="${prefix}joint_3" type="revolute">
-			<origin xyz="0 -0.18759 0.77" rpy="0 0 0"/>
+			<origin xyz="0 0 0.770" rpy="0 0 0"/>
 			<parent link="${prefix}link_2"/>
 			<child link="${prefix}link_3"/>
@@ -133,5 +134,5 @@
 		</joint>
 		<joint name="${prefix}joint_4" type="revolute">
-			<origin xyz="0.18425 0 0.1" rpy="0 0 0"/>
+			<origin xyz="0 0 0.100" rpy="0 0 0"/>
 			<parent link="${prefix}link_3"/>
 			<child link="${prefix}link_4"/>
@@ -140,5 +141,5 @@
 		</joint>
 		<joint name="${prefix}joint_5" type="revolute">
-			<origin xyz="0.55575 0 0" rpy="0 0 0"/>
+			<origin xyz="0.740 0 0" rpy="0 0 0"/>
 			<parent link="${prefix}link_4"/>
 			<child link="${prefix}link_5"/>
@@ -147,5 +148,5 @@
 		</joint>
 		<joint name="${prefix}joint_6" type="revolute">
-			<origin xyz="0.1 0 0" rpy="0 0 0"/>
+			<origin xyz="0.100 0 0" rpy="0 0 0"/>
 			<parent link="${prefix}link_5"/>
 			<child link="${prefix}link_6"/>
@@ -154,7 +155,7 @@
 		</joint>
 		<joint name="${prefix}joint_6-tool0" type="fixed">
+			<origin xyz="0 0 0" rpy="${m_pi} ${-m_pi_2} 0" />
 			<parent link="${prefix}link_6"/>
 			<child link="${prefix}tool0"/>
-			<origin xyz="0 0 0" rpy="0 0 0"/>
 		</joint>
 	</xacro:macro>
