Commit message: m430ia2p: update urdfs based on DH data. For #54 and #63.

File: fanuc_m430ia_support/urdf/m430ia2p.urdf (robot description, URDF)
Before this commit: robot fanuc_m430ia2p, 8 links, 7 joints
Joints:
- joint joint_1: origin xyz=0 0 0.2905 rpy=0 0 0 -> xyz=0 0 0.410 rpy=0 0 0
- joint joint_2: origin xyz=0 0.0845 0.1195 rpy=0 0 0 -> xyz=0 0 0 rpy=0 0 0
- joint joint_3: origin xyz=0 0 0.35 rpy=0 0 0 -> xyz=0 0 0.350 rpy=0 0 0
- joint joint_4: origin xyz=0 -0.0845 0.099 rpy=0 0 0 -> xyz=0 0 0 rpy=0 0 0
- joint joint_5: origin xyz=0 -0.042843 0.251 rpy=0 0 0 -> xyz=0 0 0.350 rpy=0 0 0
- joint joint_6: origin xyz=0 -0.052157 0.049 rpy=0 0 0 -> xyz=0 -0.095 0.065 rpy=0 0 0

File: fanuc_m430ia_support/urdf/m430ia2p_macro.xacro (robot description, xacro)
@@ -2,4 +2,5 @@
 <robot xmlns:xacro="http://ros.org/wiki/xacro">
 	<xacro:include filename="$(find fanuc_resources)/urdf/common_materials.xacro"/>
+	<xacro:include filename="$(find fanuc_resources)/urdf/common_constants.xacro"/>
 	<xacro:macro name="fanuc_m430ia2p" params="prefix">
 		<!-- links -->
@@ -112,5 +113,5 @@
 		<!-- joints -->
 		<joint name="${prefix}joint_1" type="revolute">
-			<origin xyz="0 0 0.2905" rpy="0 0 0"/>
+			<origin xyz="0 0 0.410" rpy="0 0 0"/>
 			<parent link="${prefix}base_link"/>
 			<child link="${prefix}link_1"/>
@@ -119,5 +120,5 @@
 		</joint>
 		<joint name="${prefix}joint_2" type="revolute">
-			<origin xyz="0 0.0845 0.1195" rpy="0 0 0"/>
+			<origin xyz="0 0 0" rpy="0 0 0"/>
 			<parent link="${prefix}link_1"/>
 			<child link="${prefix}link_2"/>
@@ -126,5 +127,5 @@
 		</joint>
 		<joint name="${prefix}joint_3" type="revolute">
-			<origin xyz="0 0 0.35" rpy="0 0 0"/>
+			<origin xyz="0 0 0.350" rpy="0 0 0"/>
 			<parent link="${prefix}link_2"/>
 			<child link="${prefix}link_3"/>
@@ -133,5 +134,5 @@
 		</joint>
 		<joint name="${prefix}joint_4" type="revolute">
-			<origin xyz="0 -0.0845 0.099" rpy="0 0 0"/>
+			<origin xyz="0 0 0" rpy="0 0 0"/>
 			<parent link="${prefix}link_3"/>
 			<child link="${prefix}link_4"/>
@@ -140,5 +141,5 @@
 		</joint>
 		<joint name="${prefix}joint_5" type="revolute">
-			<origin xyz="0 -0.042843 0.251" rpy="0 0 0"/>
+			<origin xyz="0 0 0.350" rpy="0 0 0"/>
 			<parent link="${prefix}link_4"/>
 			<child link="${prefix}link_5"/>
@@ -147,5 +148,5 @@
 		</joint>
 		<joint name="${prefix}joint_6" type="revolute">
-			<origin xyz="0 -0.052157 0.049" rpy="0 0 0"/>
+			<origin xyz="0 -0.095 0.065" rpy="0 0 0"/>
 			<parent link="${prefix}link_5"/>
 			<child link="${prefix}link_6"/>
@@ -154,7 +155,7 @@
 		</joint>
 		<joint name="${prefix}joint_6-tool0" type="fixed">
+			<origin xyz="0 0 0" rpy="0 0 0" />
 			<parent link="${prefix}link_6" />
 			<child link="${prefix}tool0" />
-			<origin xyz="0 0 0" rpy="0 0 0" />
 		</joint>
 	</xacro:macro>
