Commit message: m430ia2f: update urdfs based on DH data. For #54 and #63.

File: fanuc_m430ia_support/urdf/m430ia2f.urdf (robot description, URDF)
Before this commit: robot fanuc_m430ia2f, 7 links, 6 joints
Joints:
- joint joint_1: origin xyz=0 0 0.44 rpy=0 0 0 -> xyz=0 0 0.440 rpy=0 0 0
- joint joint_2: origin xyz=0 0.171 0 rpy=0 0 0 -> xyz=0 0 0 rpy=0 0 0
- joint joint_3: origin xyz=0 -0.171 0.35 rpy=0 0 0 -> xyz=0 -0.095 0.350 rpy=0 0 0
- joint joint_4: origin xyz=0 -0.06 0.55 rpy=0 0 0 -> xyz=0 0 0.550 rpy=0 0 0
- joint joint_5: origin xyz=0 -0.035 0.065 rpy=0 0 0 -> xyz=0 0 0.065 rpy=0 0 0

File: fanuc_m430ia_support/urdf/m430ia2f_macro.xacro (robot description, xacro)
@@ -2,4 +2,5 @@
 <robot xmlns:xacro="http://ros.org/wiki/xacro">
 	<xacro:include filename="$(find fanuc_resources)/urdf/common_materials.xacro"/>
+	<xacro:include filename="$(find fanuc_resources)/urdf/common_constants.xacro"/>
 	<xacro:macro name="fanuc_m430ia2f" params="prefix">
 		<!-- links -->
@@ -51,9 +52,5 @@
 		<link name="${prefix}link_3">
 			<visual>
-				<!-- coordinate origin for link_3 is not at mate centre, -->
-				<!-- so compensate (53mm dZ between link_3-link_2 mate -->
-				<!-- and coordinate origin) -->
-				<!-- origin xyz="0 0 0" rpy="0 0 0"/ -->
-				<origin xyz="0 0 0.053" rpy="0 0 0"/>
+				<origin xyz="0 0 0" rpy="0 0 0"/>
 				<geometry>
 					<mesh filename="package://fanuc_m430ia_support/meshes/m430ia2f/visual/link_3.stl"/>
@@ -62,7 +59,5 @@
 			</visual>
 			<collision>
-				<!-- see earlier comment -->
-				<!-- origin xyz="0 0 0" rpy="0 0 0"/ -->
-				<origin xyz="0 0 0.053" rpy="0 0 0"/>
+				<origin xyz="0 0 0" rpy="0 0 0"/>
 				<geometry>
 					<mesh filename="package://fanuc_m430ia_support/meshes/m430ia2f/collision/link_3.stl"/>
@@ -103,5 +98,5 @@
 		<!-- joints -->
 		<joint name="${prefix}joint_1" type="revolute">
-			<origin xyz="0 0 0.44" rpy="0 0 0"/>
+			<origin xyz="0 0 0.440" rpy="0 0 0"/>
 			<parent link="${prefix}base_link"/>
 			<child link="${prefix}link_1"/>
@@ -110,5 +105,5 @@
 		</joint>
 		<joint name="${prefix}joint_2" type="revolute">
-			<origin xyz="0 0.171 0" rpy="0 0 0"/>
+			<origin xyz="0 0 0" rpy="0 0 0"/>
 			<parent link="${prefix}link_1"/>
 			<child link="${prefix}link_2"/>
@@ -117,7 +112,5 @@
 		</joint>
 		<joint name="${prefix}joint_3" type="revolute">
-			<!-- see earlier comment -->
-			<!-- origin xyz="0 -0.171 0.403" rpy="0 0 0"/ -->
-			<origin xyz="0 -0.171 0.35" rpy="0 0 0"/>
+			<origin xyz="0 -0.095 0.350" rpy="0 0 0"/>
 			<parent link="${prefix}link_2"/>
 			<child link="${prefix}link_3"/>
@@ -126,7 +119,5 @@
 		</joint>
 		<joint name="${prefix}joint_4" type="revolute">
-			<!-- see earlier comment -->
-			<!-- origin xyz="0 -0.06 0.497" rpy="0 0 0"/ -->
-			<origin xyz="0 -0.06 0.55" rpy="0 0 0"/>
+			<origin xyz="0 0 0.550" rpy="0 0 0"/>
 			<parent link="${prefix}link_3"/>
 			<child link="${prefix}link_4"/>
@@ -135,5 +126,5 @@
 		</joint>
 		<joint name="${prefix}joint_5" type="revolute">
-			<origin xyz="0 -0.035 0.065" rpy="0 0 0"/>
+			<origin xyz="0 0 0.065" rpy="0 0 0"/>
 			<parent link="${prefix}link_4"/>
 			<child link="${prefix}link_5"/>
@@ -142,7 +133,7 @@
 		</joint>
 		<joint name="${prefix}joint_5-tool0" type="fixed">
+			<origin xyz="0 0 0" rpy="0 0 0" />
 			<parent link="${prefix}link_5"/>
 			<child link="${prefix}tool0"/>
-			<origin xyz="0 0 0" rpy="0 0 0"/>
 		</joint>
 	</xacro:macro>
