Commit message: lrmate200id: add 'base' link (transform to World Coordinates). For ros-industrial/fanuc#101.

File: fanuc_lrmate200id_support/urdf/lrmate200id.urdf (robot description, URDF)
Before this commit: robot fanuc_lrmate200id, 8 links, 7 joints
Links:
- added link base
Joints:
- added joint base_link-base: type fixed, parent base_link, child base, origin xyz=0 0 0.330 rpy=0 0 0

File: fanuc_lrmate200id_support/urdf/lrmate200id_macro.xacro (robot description, xacro)
@@ -157,4 +157,11 @@
 			<child link="${prefix}tool0" />
 		</joint>
+		<!-- ROS base_link to Fanuc World Coordinates transform -->
+		<link name="${prefix}base" />
+		<joint name="${prefix}base_link-base" type="fixed">
+			<origin xyz="0 0 0.330" rpy="0 0 0"/>
+			<parent link="${prefix}base_link"/>
+			<child link="${prefix}base"/>
+		</joint>
 	</xacro:macro>
 </robot>
