Commit message: lrmate200id: fix J3 joint limit (/7L).
According to the Operator's Manual these are the correct limits for J3 of a /7L.

File: fanuc_lrmate200id_support/urdf/lrmate200id7l_macro.xacro (robot description, xacro)
@@ -129,5 +129,5 @@
       <child link="${prefix}link_3" />
       <axis xyz="0 -1 0" />
-      <limit effort="0" lower="${radians(-149)}" upper="${radians(280)}" velocity="${radians(410)}" />
+      <limit effort="0" lower="${radians(-70)}" upper="${radians(213)}" velocity="${radians(410)}" />
     </joint>
     <joint name="${prefix}joint_4" type="revolute">

Commit message: lrmate200id: negative limit before conversion (/7L).

File: fanuc_lrmate200id_support/urdf/lrmate200id7l_macro.xacro (robot description, xacro)
@@ -136,5 +136,5 @@
       <child link="${prefix}link_4"/>
       <axis xyz="-1 0 0"/>
-      <limit effort="0" lower="-${radians(190)}" upper="${radians(190)}" velocity="${radians(550)}" />
+      <limit effort="0" lower="${radians(-190)}" upper="${radians(190)}" velocity="${radians(550)}" />
     </joint>
     <joint name="${prefix}joint_5" type="revolute">
@@ -143,5 +143,5 @@
       <child link="${prefix}link_5"/>
       <axis xyz="0 -1 0"/>
-      <limit effort="0" lower="-${radians(125)}" upper="${radians(125)}" velocity="${radians(545)}" />
+      <limit effort="0" lower="${radians(-125)}" upper="${radians(125)}" velocity="${radians(545)}" />
     </joint>
     <joint name="${prefix}joint_6" type="revolute">

Commit message: lrmate200id: fix joint names (/7L).

File: fanuc_lrmate200id_support/urdf/lrmate200id7l_macro.xacro (robot description, xacro)
@@ -161,5 +161,5 @@
     <!-- ROS-Industrial 'flange' frame: attachment point for EEF models -->
     <link name="${prefix}flange" />
-    <joint name="${prefix}joint_6-flange" type="fixed">
+    <joint name="${prefix}link_6-flange" type="fixed">
       <origin xyz="0 0 0" rpy="0 0 0" />
       <parent link="${prefix}link_6" />
@@ -168,5 +168,5 @@
     <!-- ROS-Industrial 'tool0' frame: all-zeros tool frame -->
     <link name="${prefix}tool0" />
-    <joint name="${prefix}link_6-tool0" type="fixed">
+    <joint name="${prefix}flange-tool0" type="fixed">
       <origin xyz="0 0 0" rpy="${pi} ${-pi/2.0} 0" />
       <parent link="${prefix}link_6" />

Commit message: lrmate200id: flange is parent of tool0 (/7L).
Not 'link_6'.

File: fanuc_lrmate200id_support/urdf/lrmate200id7l_macro.xacro (robot description, xacro)
@@ -170,5 +170,5 @@
     <joint name="${prefix}flange-tool0" type="fixed">
       <origin xyz="0 0 0" rpy="${pi} ${-pi/2.0} 0" />
-      <parent link="${prefix}link_6" />
+      <parent link="${prefix}flange" />
       <child link="${prefix}tool0" />
     </joint>
