Commit message: m10ia: update urdfs based on DH data. For #54 and #63.

File: fanuc_m10ia_support/urdf/m10ia.urdf (robot description, URDF)
Before this commit: robot fanuc_m10ia, 8 links, 7 joints
Joints:
- joint joint_1: origin xyz=0 0 0 rpy=0 0 0 -> xyz=0 0 0.450 rpy=0 0 0
- joint joint_2: origin xyz=0.15 -0.04 0.45 rpy=0 0 0 -> xyz=0.150 0 0 rpy=0 0 0
- joint joint_3: origin xyz=0 -0.0225 0.6 rpy=0 0 0 -> xyz=0 0 0.600 rpy=0 0 0
- joint joint_4: origin xyz=0.1805 0.0625 0.2 rpy=0 0 0 -> xyz=0 0 0.200 rpy=0 0 0
- joint joint_5: origin xyz=0.4595 -0.0565 0 rpy=0 0 0 -> xyz=0.640 0 0 rpy=0 0 0
- joint joint_6: origin xyz=0.1 0.0565 0 rpy=0 0 0 -> xyz=0.100 0 0 rpy=0 0 0
- joint joint_6-tool0: origin xyz=0 0 0 rpy=0 0 0 -> xyz=0 0 0 rpy=3.1415926535 -1.570796327 0

File: fanuc_m10ia_support/urdf/m10ia_macro.xacro (robot description, xacro)
@@ -2,9 +2,10 @@
 <robot xmlns:xacro="http://ros.org/wiki/xacro">
 	<xacro:include filename="$(find fanuc_resources)/urdf/common_materials.xacro"/>
+	<xacro:include filename="$(find fanuc_resources)/urdf/common_constants.xacro"/>
 	<xacro:macro name="fanuc_m10ia" params="prefix">
 		<!-- links -->
 		<link name="${prefix}base_link">
 			<visual>
-				<origin xyz="0 0 0" rpy="-1.578 0 0"/>
+				<origin xyz="0 0 0" rpy="0 0 0"/>
 				<geometry>
 					<mesh filename="package://fanuc_m10ia_support/meshes/m10ia/visual/base_link.stl"/>
@@ -13,5 +14,5 @@
 			</visual>
 			<collision>
-				<origin xyz="0 0 0" rpy="-1.578 0 0"/>
+				<origin xyz="0 0 0" rpy="0 0 0"/>
 				<geometry>
 					<mesh filename="package://fanuc_m10ia_support/meshes/m10ia/collision/base_link.stl"/>
@@ -112,5 +113,5 @@
 		<!-- joints -->
 		<joint name="${prefix}joint_1" type="revolute">
-			<origin xyz="0 0 0" rpy="0 0 0"/>
+			<origin xyz="0 0 0.450" rpy="0 0 0"/>
 			<parent link="${prefix}base_link"/>
 			<child link="${prefix}link_1"/>
@@ -119,5 +120,5 @@
 		</joint>
 		<joint name="${prefix}joint_2" type="revolute">
-			<origin xyz="0.15 -0.04 0.45" rpy="0 0 0"/>
+			<origin xyz="0.150 0 0" rpy="0 0 0"/>
 			<parent link="${prefix}link_1"/>
 			<child link="${prefix}link_2"/>
@@ -126,5 +127,5 @@
 		</joint>
 		<joint name="${prefix}joint_3" type="revolute">
-			<origin xyz="0 -0.0225 0.6" rpy="0 0 0"/>
+			<origin xyz="0 0 0.600" rpy="0 0 0"/>
 			<parent link="${prefix}link_2"/>
 			<child link="${prefix}link_3"/>
@@ -133,5 +134,5 @@
 		</joint>
 		<joint name="${prefix}joint_4" type="revolute">
-			<origin xyz="0.1805 0.0625 0.2" rpy="0 0 0"/>
+			<origin xyz="0 0 0.200" rpy="0 0 0"/>
 			<parent link="${prefix}link_3"/>
 			<child link="${prefix}link_4"/>
@@ -140,5 +141,5 @@
 		</joint>
 		<joint name="${prefix}joint_5" type="revolute">
-			<origin xyz="0.4595 -0.0565 0" rpy="0 0 0"/>
+			<origin xyz="0.640 0 0" rpy="0 0 0"/>
 			<parent link="${prefix}link_4"/>
 			<child link="${prefix}link_5"/>
@@ -147,5 +148,5 @@
 		</joint>
 		<joint name="${prefix}joint_6" type="revolute">
-			<origin xyz="0.1 0.0565 0" rpy="0 0 0"/>
+			<origin xyz="0.100 0 0" rpy="0 0 0"/>
 			<parent link="${prefix}link_5"/>
 			<child link="${prefix}link_6"/>
@@ -154,7 +155,7 @@
 		</joint>
 		<joint name="${prefix}joint_6-tool0" type="fixed">
+			<origin xyz="0 0 0" rpy="${m_pi} ${-m_pi_2} 0" />
 			<parent link="${prefix}link_6"/>
 			<child link="${prefix}tool0"/>
-			<origin xyz="0 0 0" rpy="0 0 0"/>
 		</joint>
 	</xacro:macro>

Commit message: support: add 'base' link (transform to World Coordinates). Fix #101.
This should not affect existing kinematic plugins or MoveIt configurations:

 - the link is not part of the main kinematic chain
 - the transform is implemented as a fixed joint

File: fanuc_m10ia_support/urdf/m10ia.urdf (robot description, URDF)
Before this commit: robot fanuc_m10ia, 8 links, 7 joints
Links:
- added link base
Joints:
- added joint base_link-base: type fixed, parent base_link, child base, origin xyz=0 0 0.450 rpy=0 0 0

File: fanuc_m10ia_support/urdf/m10ia_macro.xacro (robot description, xacro)
@@ -159,4 +159,11 @@
 			<child link="${prefix}tool0"/>
 		</joint>
+		<!-- ROS base_link to Fanuc World Coordinates transform -->
+		<link name="${prefix}base" />
+		<joint name="${prefix}base_link-base" type="fixed">
+			<origin xyz="0 0 0.450" rpy="0 0 0"/>
+			<parent link="${prefix}base_link"/>
+			<child link="${prefix}base"/>
+		</joint>
 	</xacro:macro>
 </robot>

File: fanuc_m16ib_support/urdf/m16ib20.urdf (robot description, URDF)
Before this commit: robot fanuc_m16ib20, 8 links, 7 joints
Links:
- added link base
Joints:
- added joint base_link-base: type fixed, parent base_link, child base, origin xyz=0 0 0.525 rpy=0 0 0

File: fanuc_m16ib_support/urdf/m16ib20_macro.xacro (robot description, xacro)
@@ -159,4 +159,11 @@
 			<child link="${prefix}tool0"/>
 		</joint>
+		<!-- ROS base_link to Fanuc World Coordinates transform -->
+		<link name="${prefix}base" />
+		<joint name="${prefix}base_link-base" type="fixed">
+			<origin xyz="0 0 0.525" rpy="0 0 0"/>
+			<parent link="${prefix}base_link"/>
+			<child link="${prefix}base"/>
+		</joint>
 	</xacro:macro>
 </robot>

File: fanuc_m430ia_support/urdf/m430ia2f.urdf (robot description, URDF)
Before this commit: robot fanuc_m430ia2f, 7 links, 6 joints
Links:
- added link base
Joints:
- added joint base_link-base: type fixed, parent base_link, child base, origin xyz=0 0 0.440 rpy=0 0 0

File: fanuc_m430ia_support/urdf/m430ia2f_macro.xacro (robot description, xacro)
@@ -137,4 +137,11 @@
 			<child link="${prefix}tool0"/>
 		</joint>
+		<!-- ROS base_link to Fanuc World Coordinates transform -->
+		<link name="${prefix}base" />
+		<joint name="${prefix}base_link-base" type="fixed">
+			<origin xyz="0 0 0.440" rpy="0 0 0"/>
+			<parent link="${prefix}base_link"/>
+			<child link="${prefix}base"/>
+		</joint>
 	</xacro:macro>
 </robot>

File: fanuc_m430ia_support/urdf/m430ia2p.urdf (robot description, URDF)
Before this commit: robot fanuc_m430ia2p, 8 links, 7 joints
Links:
- added link base
Joints:
- added joint base_link-base: type fixed, parent base_link, child base, origin xyz=0 0 0.410 rpy=0 0 0

File: fanuc_m430ia_support/urdf/m430ia2p_macro.xacro (robot description, xacro)
@@ -159,4 +159,11 @@
 			<child link="${prefix}tool0" />
 		</joint>
+		<!-- ROS base_link to Fanuc World Coordinates transform -->
+		<link name="${prefix}base" />
+		<joint name="${prefix}base_link-base" type="fixed">
+			<origin xyz="0 0 0.410" rpy="0 0 0"/>
+			<parent link="${prefix}base_link"/>
+			<child link="${prefix}base"/>
+		</joint>
 	</xacro:macro>
 </robot>
