Commit message: Fix axis 6 wrong direction in M-710iC definition (ros-industrial/fanuc_experimental#28)

File: fanuc_m710ic_support/urdf/m710ic50.urdf (robot description, URDF)
Before this commit: robot fanuc_m710ic50, 9 links, 8 joints
Joints:
- joint joint_6: axis 1 0 0 -> -1 0 0

File: fanuc_m710ic_support/urdf/m710ic50_macro.xacro (robot description, xacro)
@@ -149,5 +149,5 @@
       <parent link="${prefix}link_5"/>
       <child link="${prefix}link_6"/>
-      <axis xyz="1 0 0"/>
+      <axis xyz="-1 0 0"/>
       <limit effort="0" lower="-6.2831" upper="6.2831" velocity="6.1959" />
     </joint>
