Commit message: m710ic50: update joint limits based on ctrlr data.

File: fanuc_m710ic_support/urdf/m710ic50_macro.xacro (robot description, xacro)
@@ -115,5 +115,5 @@
       <child link="${prefix}link_1" />
       <axis xyz="0 0 1" />
-      <limit effort="0" lower="-3.1415" upper="3.1415" velocity="3.05" />
+      <limit effort="0" lower="-3.1415" upper="3.1415" velocity="3.0543" />
     </joint>
     <joint name="${prefix}joint_2" type="revolute">
@@ -122,5 +122,5 @@
       <child link="${prefix}link_2" />
       <axis xyz="0 1 0" />
-      <limit effort="0" lower="-1.57" upper="2.35" velocity="3.05" />
+      <limit effort="0" lower="-1.5707" upper="2.3561" velocity="3.0543" />
     </joint>
     <joint name="${prefix}joint_3" type="revolute">
@@ -129,5 +129,5 @@
       <child link="${prefix}link_3" />
       <axis xyz="0 -1 0" />
-      <limit effort="0" lower="-2.79" upper="4.88" velocity="3.05" />
+      <limit effort="0" lower="-2.7925" upper="4.8869" velocity="3.0543" />
     </joint>
     <joint name="${prefix}joint_4" type="revolute">
@@ -136,5 +136,5 @@
       <child link="${prefix}link_4"/>
       <axis xyz="-1 0 0"/>
-      <limit effort="0" lower="-6.2830" upper="6.2830" velocity="4.36" />
+      <limit effort="0" lower="-6.2830" upper="6.2830" velocity="4.3633" />
     </joint>
     <joint name="${prefix}joint_5" type="revolute">
@@ -143,5 +143,5 @@
       <child link="${prefix}link_5"/>
       <axis xyz="0 -1 0"/>
-      <limit effort="0" lower="-2.18" upper="2.18" velocity="4.36" />
+      <limit effort="0" lower="-2.1816" upper="2.1816" velocity="4.3633" />
     </joint>
     <joint name="${prefix}joint_6" type="revolute">
@@ -150,5 +150,5 @@
       <child link="${prefix}link_6"/>
       <axis xyz="1 0 0"/>
-      <limit effort="0" lower="-6.285" upper="6.285" velocity="6.20" />
+      <limit effort="0" lower="-6.2831" upper="6.2831" velocity="6.1959" />
     </joint>
     <joint name="${prefix}joint_6-tool0" type="fixed">

Commit message: support: add 'flange' frame.
Ref: ros-industrial/fanuc@aba7f6c97dfee493a92e4edf4c2013eb303355d7.

File: fanuc_m710ic_support/urdf/m710ic50_macro.xacro (robot description, xacro)
@@ -3,4 +3,5 @@
   <xacro:include filename="$(find fanuc_resources)/urdf/common_materials.xacro"/>
   <xacro:macro name="fanuc_m710ic50" params="prefix">
+    <!-- links: main serial chain -->
     <link name="${prefix}base_link">
       <visual>
@@ -108,5 +109,5 @@
       </collision>
     </link>
-    <link name="${prefix}tool0" />
+    <!-- joints: main serial chain -->
     <joint name="${prefix}joint_1" type="revolute">
       <origin xyz="0 0 0.565" rpy="0 0 0" />
@@ -151,10 +152,5 @@
       <limit effort="0" lower="-6.2831" upper="6.2831" velocity="6.1959" />
     </joint>
-    <joint name="${prefix}joint_6-tool0" type="fixed">
-      <origin xyz="0 0 0" rpy="${pi} ${-pi/2.0} 0" />
-      <parent link="${prefix}link_6" />
-      <child link="${prefix}tool0" />
-    </joint>
-    <!-- ROS base_link to Fanuc World Coordinates transform -->
+    <!-- ROS-Industrial 'base' frame: base_link to Fanuc World Coordinates transform -->
     <link name="${prefix}base" />
     <joint name="${prefix}base_link-base" type="fixed">
@@ -163,4 +159,18 @@
       <child link="${prefix}base"/>
     </joint>
+    <!-- ROS-Industrial 'flange' frame: attachment point for EEF models -->
+    <link name="${prefix}flange" />
+    <joint name="${prefix}joint_6-flange" type="fixed">
+      <origin xyz="0 0 0" rpy="0 0 0" />
+      <parent link="${prefix}link_6" />
+      <child link="${prefix}flange" />
+    </joint>
+    <!-- ROS-Industrial 'tool0' frame: all-zeros tool frame -->
+    <link name="${prefix}tool0" />
+    <joint name="${prefix}link_6-tool0" type="fixed">
+      <origin xyz="0 0 0" rpy="${pi} ${-pi/2.0} 0" />
+      <parent link="${prefix}link_6" />
+      <child link="${prefix}tool0" />
+    </joint>
   </xacro:macro>
 </robot>
