Commit message: support: use Jade+ xacro 'pi' constant instead of redefining it ourselves.

File: fanuc_lrmate200ic_support/urdf/lrmate200ic5f_macro.xacro (robot description, xacro)
@@ -131,5 +131,5 @@
     </joint>
     <joint name="${prefix}joint_5-tool0" type="fixed">
-      <origin xyz="0 0 0" rpy="${m_pi} ${-m_pi_2} 0" />
+      <origin xyz="0 0 0" rpy="${pi} ${-pi/2.0} 0" />
       <parent link="${prefix}link_5" />
       <child link="${prefix}tool0" />

File: fanuc_lrmate200ic_support/urdf/lrmate200ic5h_macro.xacro (robot description, xacro)
@@ -131,5 +131,5 @@
     </joint>
     <joint name="${prefix}joint_5-tool0" type="fixed">
-      <origin xyz="0 0 0" rpy="${m_pi} ${-m_pi_2} 0" />
+      <origin xyz="0 0 0" rpy="${pi} ${-pi/2.0} 0" />
       <parent link="${prefix}link_5" />
       <child link="${prefix}tool0" />

File: fanuc_lrmate200ic_support/urdf/lrmate200ic5hs_macro.xacro (robot description, xacro)
@@ -131,5 +131,5 @@
     </joint>
     <joint name="${prefix}joint_5-tool0" type="fixed">
-      <origin xyz="0 0 0" rpy="${m_pi} ${-m_pi_2} 0" />
+      <origin xyz="0 0 0" rpy="${pi} ${-pi/2.0} 0" />
       <parent link="${prefix}link_5" />
       <child link="${prefix}tool0" />

File: fanuc_lrmate200ic_support/urdf/lrmate200ic5l_macro.xacro (robot description, xacro)
@@ -153,5 +153,5 @@
     </joint>
     <joint name="${prefix}joint_6-tool0" type="fixed">
-      <origin xyz="0 0 0" rpy="${m_pi} ${-m_pi_2} 0" />
+      <origin xyz="0 0 0" rpy="${pi} ${-pi/2.0} 0" />
       <parent link="${prefix}link_6" />
       <child link="${prefix}tool0" />

File: fanuc_lrmate200ic_support/urdf/lrmate200ic_macro.xacro (robot description, xacro)
@@ -153,5 +153,5 @@
     </joint>
     <joint name="${prefix}joint_6-tool0" type="fixed">
-      <origin xyz="0 0 0" rpy="${m_pi} ${-m_pi_2} 0" />
+      <origin xyz="0 0 0" rpy="${pi} ${-pi/2.0} 0" />
       <parent link="${prefix}link_6" />
       <child link="${prefix}tool0" />

File: fanuc_m10ia_support/urdf/m10ia7l_macro.xacro (robot description, xacro)
@@ -155,5 +155,5 @@
     </joint>
     <joint name="${prefix}joint_6-tool0" type="fixed">
-      <origin xyz="0 0 0" rpy="${m_pi} ${-m_pi_2} 0" />
+      <origin xyz="0 0 0" rpy="${pi} ${-pi/2.0} 0" />
       <parent link="${prefix}link_6"/>
       <child link="${prefix}tool0"/>

File: fanuc_m10ia_support/urdf/m10ia_macro.xacro (robot description, xacro)
@@ -155,5 +155,5 @@
     </joint>
     <joint name="${prefix}joint_6-tool0" type="fixed">
-      <origin xyz="0 0 0" rpy="${m_pi} ${-m_pi_2} 0" />
+      <origin xyz="0 0 0" rpy="${pi} ${-pi/2.0} 0" />
       <parent link="${prefix}link_6"/>
       <child link="${prefix}tool0"/>

File: fanuc_m16ib_support/urdf/m16ib20_macro.xacro (robot description, xacro)
@@ -155,5 +155,5 @@
     </joint>
     <joint name="${prefix}joint_6-tool0" type="fixed">
-      <origin xyz="0 0 0" rpy="${m_pi} ${-m_pi_2} 0" />
+      <origin xyz="0 0 0" rpy="${pi} ${-pi/2.0} 0" />
       <parent link="${prefix}link_6"/>
       <child link="${prefix}tool0"/>

File: fanuc_m20ia_support/urdf/m20ia10l_macro.xacro (robot description, xacro)
@@ -155,5 +155,5 @@
     </joint>
     <joint name="${prefix}joint_6-tool0" type="fixed">
-      <origin xyz="0 0 0" rpy="${m_pi} ${-m_pi_2} 0" />
+      <origin xyz="0 0 0" rpy="${pi} ${-pi/2.0} 0" />
       <parent link="${prefix}link_6"/>
       <child link="${prefix}tool0"/>

File: fanuc_m20ia_support/urdf/m20ia_macro.xacro (robot description, xacro)
@@ -155,5 +155,5 @@
     </joint>
     <joint name="${prefix}joint_6-tool0" type="fixed">
-      <origin xyz="0 0 0" rpy="${m_pi} ${-m_pi_2} 0" />
+      <origin xyz="0 0 0" rpy="${pi} ${-pi/2.0} 0" />
       <parent link="${prefix}link_6"/>
       <child link="${prefix}tool0"/>
