Commit message: support: add 'flange' frame.
The 'flange' frame is intended to function as an 'attachment point' for
EEF xacros. In order to easily swap robot models, it is beneficial for
such attachment points -- typically the last link in a robot xacro -- to
have a consistent orientation.

'flange' is defined as always having x+ pointing out of the (physical)
flange link. For robots that happen to have the link-local coordinate
frame of their last link in their zero pose already aligned with REP-103
conventions (x+ forward, y+ left, z+ up), 'flange' will be an identity
transform. In other cases, 'flange' includes appropriate rotations to
orient x+ such that it again follows the above described convention.

Note that the above does not mean that 'flange' will *always* be world
aligned, only that x+ will always point away from the (physical) flange /
last link of the robot model. Rotations and translations will impact
'flange's pose just as they do other robot links.

It's sibling frame, 'tool0', is similar, but this frame is *always*
located and oriented such that it corresponds to whatever is configured on
the robot controller as an 'all zeros' tool frame.

Both 'tool0' and 'flange' are to be considered immutable frames, and are
not intended to be changed or updated by consumers of xacro macros
including them.

File: fanuc_m430ia_support/urdf/m430ia2p_macro.xacro (robot description, xacro)
@@ -3,5 +3,5 @@
   <xacro:include filename="$(find fanuc_resources)/urdf/common_materials.xacro"/>
   <xacro:macro name="fanuc_m430ia2p" params="prefix">
-    <!-- links -->
+    <!-- links: main serial chain -->
     <link name="${prefix}base_link">
       <visual>
@@ -109,6 +109,5 @@
       </collision>
     </link>
-    <link name="${prefix}tool0" />
-    <!-- joints -->
+    <!-- joints: main serial chain -->
     <joint name="${prefix}joint_1" type="revolute">
       <origin xyz="0 0 0.410" rpy="0 0 0"/>
@@ -153,10 +152,5 @@
       <limit lower="-4.71" upper="4.71" effort="0" velocity="12.57"/>
     </joint>
-    <joint name="${prefix}joint_6-tool0" type="fixed">
-      <origin xyz="0 0 0" rpy="0 0 0" />
-      <parent link="${prefix}link_6" />
-      <child link="${prefix}tool0" />
-    </joint>
-    <!-- ROS base_link to Fanuc World Coordinates transform -->
+    <!-- ROS-Industrial 'base' frame: base_link to Fanuc World Coordinates transform -->
     <link name="${prefix}base" />
     <joint name="${prefix}base_link-base" type="fixed">
@@ -165,4 +159,18 @@
       <child link="${prefix}base"/>
     </joint>
+    <!-- ROS-Industrial 'flange' frame: attachment point for EEF models -->
+    <link name="${prefix}flange" />
+    <joint name="${prefix}joint_6-flange" type="fixed">
+      <origin xyz="0 0 0" rpy="0 ${-pi/2.0} 0" />
+      <parent link="${prefix}link_6" />
+      <child link="${prefix}flange" />
+    </joint>
+    <!-- ROS-Industrial 'tool0' frame: all-zeros tool frame -->
+    <link name="${prefix}tool0" />
+    <joint name="${prefix}link_6-tool0" type="fixed">
+      <origin xyz="0 0 0" rpy="0 0 0" />
+      <parent link="${prefix}link_6" />
+      <child link="${prefix}tool0" />
+    </joint>
   </xacro:macro>
 </robot>
