Commit message: support: add 'flange' frame.
Ref: ros-industrial/fanuc@aba7f6c97dfee493a92e4edf4c2013eb303355d7.

File: fanuc_m20ib_support/urdf/m20ib25_macro.xacro (robot description, xacro)
@@ -3,5 +3,5 @@
   <xacro:include filename="$(find fanuc_resources)/urdf/common_materials.xacro"/>
   <xacro:macro name="fanuc_m20ib25" params="prefix">
-    <!-- links -->
+    <!-- links: main serial chain -->
     <link name="${prefix}base_link">
       <visual>
@@ -109,6 +109,5 @@
       </collision>
     </link>
-    <link name="${prefix}tool0"/>
-    <!-- joints -->
+    <!-- joints: main serial chain -->
     <joint name="${prefix}joint_1" type="revolute">
       <origin xyz="0 0 0.650" rpy="0 0 0"/>
@@ -153,10 +152,5 @@
       <limit lower="${radians(-270)}" upper="${radians(270)}" effort="0" velocity="${radians(880)}" />
     </joint>
-    <joint name="${prefix}joint_6-tool0" type="fixed">
-      <origin xyz="0 0 0" rpy="${pi} ${-pi/2.0} 0" />
-      <parent link="${prefix}link_6"/>
-      <child link="${prefix}tool0"/>
-    </joint>
-    <!-- ROS base_link to Fanuc World Coordinates transform -->
+    <!-- ROS-Industrial 'base' frame: base_link to Fanuc World Coordinates transform -->
     <link name="${prefix}base" />
     <joint name="${prefix}base_link-base" type="fixed">
@@ -165,4 +159,18 @@
       <child link="${prefix}base"/>
     </joint>
+    <!-- ROS-Industrial 'flange' frame: attachment point for EEF models -->
+    <link name="${prefix}flange" />
+    <joint name="${prefix}joint_6-flange" type="fixed">
+      <origin xyz="0 0 0" rpy="0 0 0" />
+      <parent link="${prefix}link_6" />
+      <child link="${prefix}flange" />
+    </joint>
+    <!-- ROS-Industrial 'tool0' frame: all-zeros tool frame -->
+    <link name="${prefix}tool0" />
+    <joint name="${prefix}link_6-tool0" type="fixed">
+      <origin xyz="0 0 0" rpy="${pi} ${-pi/2.0} 0" />
+      <parent link="${prefix}link_6" />
+      <child link="${prefix}tool0" />
+    </joint>
   </xacro:macro>
 </robot>
