Commit message: support: use Jade+ xacro 'pi' constant instead of redefining it ourselves.
Ref: ros-industrial/fanuc#209.

File: fanuc_m900ib_support/urdf/m900ib700_macro.xacro (robot description, xacro)
@@ -162,5 +162,5 @@
     </joint>
     <joint name="${prefix}joint_6-tool0" type="fixed">
-      <origin xyz="0 0 0" rpy="${m_pi} ${-m_pi_2} 0" />
+      <origin xyz="0 0 0" rpy="${pi} ${-pi/2.0} 0" />
       <parent link="${prefix}link_6"/>
       <child link="${prefix}tool0"/>

Commit message: m900ib: remove use of deprecated constant.
Ref: 7e148662106499ab3405c630dfb9339b1af0171d.

File: fanuc_m900ib_support/urdf/m900ib700_macro.xacro (robot description, xacro)
@@ -246,5 +246,5 @@
     <link name="${prefix}balancer_right">
       <visual>
-        <origin xyz="0 0 0" rpy="0 0 ${m_pi}"/>
+        <origin xyz="0 0 0" rpy="0 0 ${pi}"/>
         <geometry>
           <mesh filename="package://fanuc_m900ib_support/meshes/m900ib700/visual/balancer.stl"/>
@@ -253,5 +253,5 @@
       </visual>
       <collision>
-        <origin xyz="0 0 0" rpy="0 0 ${m_pi}"/>
+        <origin xyz="0 0 0" rpy="0 0 ${pi}"/>
         <geometry>
           <mesh filename="package://fanuc_m900ib_support/meshes/m900ib700/collision/balancer.stl"/>
@@ -261,5 +261,5 @@
     <link name="${prefix}piston_right">
       <visual>
-        <origin xyz="0 0 0" rpy="0 0 ${m_pi}"/>
+        <origin xyz="0 0 0" rpy="0 0 ${pi}"/>
         <geometry>
           <mesh filename="package://fanuc_m900ib_support/meshes/m900ib700/visual/piston.stl"/>
@@ -268,5 +268,5 @@
       </visual>
       <collision>
-        <origin xyz="0 0 0" rpy="0 0 ${m_pi}"/>
+        <origin xyz="0 0 0" rpy="0 0 ${pi}"/>
         <geometry>
           <mesh filename="package://fanuc_m900ib_support/meshes/m900ib700/collision/piston.stl"/>

Commit message: support: add 'flange' frame.
Ref: ros-industrial/fanuc@aba7f6c97dfee493a92e4edf4c2013eb303355d7.

File: fanuc_m900ib_support/urdf/m900ib700_macro.xacro (robot description, xacro)
@@ -10,5 +10,5 @@
   <!-- base macro -->
   <xacro:macro name="fanuc_m900ib700_base" params="prefix has_plinks has_balancers has_fl_pockets">
-    <!-- links -->
+    <!-- links: main serial chain -->
     <link name="${prefix}base_link">
       <visual>
@@ -116,6 +116,5 @@
       </collision>
     </link>
-    <link name="${prefix}tool0" />
-    <!-- joints -->
+    <!-- joints: main serial chain -->
     <joint name="${prefix}joint_1" type="revolute">
       <origin xyz="0 0 0.940" rpy="0 0 0"/>
@@ -160,9 +159,4 @@
       <limit effort="0" lower="-6.2831" upper="6.2831" velocity="2.7925"/>
     </joint>
-    <joint name="${prefix}joint_6-tool0" type="fixed">
-      <origin xyz="0 0 0" rpy="${pi} ${-pi/2.0} 0" />
-      <parent link="${prefix}link_6"/>
-      <child link="${prefix}tool0"/>
-    </joint>
     <!-- parallel bar linkage -->
     <xacro:if value="${has_plinks}">
@@ -326,5 +320,5 @@
     </joint>
     </xacro:if>
-    <!-- ROS base_link to Fanuc World Coordinates transform -->
+    <!-- ROS-Industrial 'base' frame: base_link to Fanuc World Coordinates transform -->
     <link name="${prefix}base" />
     <joint name="${prefix}base_link-base" type="fixed">
@@ -333,4 +327,18 @@
       <child link="${prefix}base"/>
     </joint>
+    <!-- ROS-Industrial 'flange' frame: attachment point for EEF models -->
+    <link name="${prefix}flange" />
+    <joint name="${prefix}joint_6-flange" type="fixed">
+      <origin xyz="0 0 0" rpy="0 0 0" />
+      <parent link="${prefix}link_6" />
+      <child link="${prefix}flange" />
+    </joint>
+    <!-- ROS-Industrial 'tool0' frame: all-zeros tool frame -->
+    <link name="${prefix}tool0" />
+    <joint name="${prefix}link_6-tool0" type="fixed">
+      <origin xyz="0 0 0" rpy="${pi} ${-pi/2.0} 0" />
+      <parent link="${prefix}link_6" />
+      <child link="${prefix}tool0" />
+    </joint>
   </xacro:macro>
 </robot>
