Commit message: support: use Jade+ xacro 'pi' constant instead of redefining it ourselves.
Ref: ros-industrial/fanuc#209.

File: fanuc_r1000ia_support/urdf/r1000ia80f_macro.xacro (robot description, xacro)
@@ -155,5 +155,5 @@
     </joint>
     <joint name="${prefix}joint_6-tool0" type="fixed">
-      <origin xyz="0 0 0" rpy="${m_pi} ${-m_pi_2} 0" />
+      <origin xyz="0 0 0" rpy="${pi} ${-pi/2.0} 0" />
       <parent link="${prefix}link_6"/>
       <child link="${prefix}tool0"/>

Commit message: support: add 'flange' frame.
Ref: ros-industrial/fanuc@aba7f6c97dfee493a92e4edf4c2013eb303355d7.

File: fanuc_r1000ia_support/urdf/r1000ia80f_macro.xacro (robot description, xacro)
@@ -3,5 +3,5 @@
   <xacro:include filename="$(find fanuc_resources)/urdf/common_materials.xacro"/>
   <xacro:macro name="fanuc_r1000ia80f" params="prefix">
-    <!-- links -->
+    <!-- links: main serial chain -->
     <link name="${prefix}base_link">
       <visual>
@@ -109,6 +109,5 @@
       </collision>
     </link>
-    <link name="${prefix}tool0"/>
-    <!-- joints -->
+    <!-- joints: main serial chain -->
     <joint name="${prefix}joint_1" type="revolute">
       <origin xyz="0 0 0.450" rpy="0 0 0"/>
@@ -153,10 +152,5 @@
       <limit lower="-6.2831" upper="6.2831" effort="0" velocity="6.1086"/>
     </joint>
-    <joint name="${prefix}joint_6-tool0" type="fixed">
-      <origin xyz="0 0 0" rpy="${pi} ${-pi/2.0} 0" />
-      <parent link="${prefix}link_6"/>
-      <child link="${prefix}tool0"/>
-    </joint>
-    <!-- ROS base_link to Fanuc World Coordinates transform -->
+    <!-- ROS-Industrial 'base' frame: base_link to Fanuc World Coordinates transform -->
     <link name="${prefix}base" />
     <joint name="${prefix}base_link-base" type="fixed">
@@ -165,4 +159,18 @@
       <child link="${prefix}base"/>
     </joint>
+    <!-- ROS-Industrial 'flange' frame: attachment point for EEF models -->
+    <link name="${prefix}flange" />
+    <joint name="${prefix}joint_6-flange" type="fixed">
+      <origin xyz="0 0 0" rpy="0 0 0" />
+      <parent link="${prefix}link_6" />
+      <child link="${prefix}flange" />
+    </joint>
+    <!-- ROS-Industrial 'tool0' frame: all-zeros tool frame -->
+    <link name="${prefix}tool0" />
+    <joint name="${prefix}link_6-tool0" type="fixed">
+      <origin xyz="0 0 0" rpy="${pi} ${-pi/2.0} 0" />
+      <parent link="${prefix}link_6" />
+      <child link="${prefix}tool0" />
+    </joint>
   </xacro:macro>
 </robot>
