Commit message: support: use Jade+ xacro 'pi' constant instead of redefining it ourselves.
Ref: ros-industrial/fanuc#209.

File: fanuc_cr35ia_support/urdf/cr35ia_macro.xacro (robot description, xacro)
@@ -157,5 +157,5 @@
     </joint>
     <joint name="${prefix}joint_6-tool0" type="fixed">
-      <origin xyz="0 0 0" rpy="${m_pi} ${-m_pi_2} 0" />
+      <origin xyz="0 0 0" rpy="${pi} ${-pi/2.0} 0" />
       <parent link="${prefix}link_6"/>
       <child link="${prefix}tool0"/>

Commit message: support: add 'flange' frame.
Ref: ros-industrial/fanuc@aba7f6c97dfee493a92e4edf4c2013eb303355d7.

File: fanuc_cr35ia_support/urdf/cr35ia_macro.xacro (robot description, xacro)
@@ -3,5 +3,5 @@
   <xacro:include filename="$(find fanuc_resources)/urdf/common_materials.xacro"/>
   <xacro:macro name="fanuc_cr35ia" params="prefix">
-    <!-- links -->
+    <!-- links: main serial chain -->
     <link name="${prefix}base_link">
       <visual>
@@ -109,6 +109,5 @@
       </collision>
     </link>
-    <link name="${prefix}tool0"/>
-    <!-- joints -->
+    <!-- joints: main serial chain -->
     <joint name="${prefix}joint_1" type="revolute">
       <origin xyz="0 0 1.180" rpy="0 0 0"/>
@@ -155,10 +154,5 @@
       <limit lower="-7.8539" upper="7.8539" effort="0" velocity="6.9813"/>
     </joint>
-    <joint name="${prefix}joint_6-tool0" type="fixed">
-      <origin xyz="0 0 0" rpy="${pi} ${-pi/2.0} 0" />
-      <parent link="${prefix}link_6"/>
-      <child link="${prefix}tool0"/>
-    </joint>
-    <!-- ROS base_link to Fanuc World Coordinates transform -->
+    <!-- ROS-Industrial 'base' frame: base_link to Fanuc World Coordinates transform -->
     <link name="${prefix}base" />
     <joint name="${prefix}base_link-base" type="fixed">
@@ -167,4 +161,18 @@
       <child link="${prefix}base"/>
     </joint>
+    <!-- ROS-Industrial 'flange' frame: attachment point for EEF models -->
+    <link name="${prefix}flange" />
+    <joint name="${prefix}joint_6-flange" type="fixed">
+      <origin xyz="0 0 0" rpy="0 0 0" />
+      <parent link="${prefix}link_6" />
+      <child link="${prefix}flange" />
+    </joint>
+    <!-- ROS-Industrial 'tool0' frame: all-zeros tool frame -->
+    <link name="${prefix}tool0" />
+    <joint name="${prefix}link_6-tool0" type="fixed">
+      <origin xyz="0 0 0" rpy="${pi} ${-pi/2.0} 0" />
+      <parent link="${prefix}link_6" />
+      <child link="${prefix}tool0" />
+    </joint>
   </xacro:macro>
 </robot>

Commit message: support: make flange parent of tool0.
In preparation for complying with 'Coordinate Frames for Serial Industrial
Manipulators'.

File: fanuc_cr35ia_support/urdf/cr35ia_macro.xacro (robot description, xacro)
@@ -172,5 +172,5 @@
     <joint name="${prefix}link_6-tool0" type="fixed">
       <origin xyz="0 0 0" rpy="${pi} ${-pi/2.0} 0" />
-      <parent link="${prefix}link_6" />
+      <parent link="${prefix}flange" />
       <child link="${prefix}tool0" />
     </joint>

File: fanuc_cr7ia_support/urdf/cr7ia_macro.xacro (robot description, xacro)
@@ -170,5 +170,5 @@
     <joint name="${prefix}link_6-tool0" type="fixed">
       <origin xyz="0 0 0" rpy="${pi} ${-pi/2.0} 0" />
-      <parent link="${prefix}link_6" />
+      <parent link="${prefix}flange" />
       <child link="${prefix}tool0" />
     </joint>

File: fanuc_cr7ia_support/urdf/cr7ial_macro.xacro (robot description, xacro)
@@ -170,5 +170,5 @@
     <joint name="${prefix}link_6-tool0" type="fixed">
       <origin xyz="0 0 0" rpy="${pi} ${-pi/2.0} 0" />
-      <parent link="${prefix}link_6" />
+      <parent link="${prefix}flange" />
       <child link="${prefix}tool0" />
     </joint>

File: fanuc_lrmate200i_support/urdf/lrmate200i_macro.xacro (robot description, xacro)
@@ -170,5 +170,5 @@
     <joint name="${prefix}link_6-tool0" type="fixed">
       <origin xyz="0 0 0" rpy="${pi} ${-pi/2.0} 0" />
-      <parent link="${prefix}link_6" />
+      <parent link="${prefix}flange" />
       <child link="${prefix}tool0" />
     </joint>

File: fanuc_lrmate200ib_support/urdf/lrmate200ib3l_macro.xacro (robot description, xacro)
@@ -170,5 +170,5 @@
     <joint name="${prefix}link_6-tool0" type="fixed">
       <origin xyz="0 0 0" rpy="${pi} ${-pi/2.0} 0" />
-      <parent link="${prefix}link_6" />
+      <parent link="${prefix}flange" />
       <child link="${prefix}tool0" />
     </joint>

File: fanuc_lrmate200ib_support/urdf/lrmate200ib_macro.xacro (robot description, xacro)
@@ -170,5 +170,5 @@
     <joint name="${prefix}link_6-tool0" type="fixed">
       <origin xyz="0 0 0" rpy="${pi} ${-pi/2.0} 0" />
-      <parent link="${prefix}link_6" />
+      <parent link="${prefix}flange" />
       <child link="${prefix}tool0" />
     </joint>

File: fanuc_lrmate200ic_support/urdf/lrmate200ic5f_macro.xacro (robot description, xacro)
@@ -148,5 +148,5 @@
     <joint name="${prefix}link_5-tool0" type="fixed">
       <origin xyz="0 0 0" rpy="${pi} ${-pi/2.0} 0" />
-      <parent link="${prefix}link_5" />
+      <parent link="${prefix}flange" />
       <child link="${prefix}tool0" />
     </joint>

File: fanuc_lrmate200ic_support/urdf/lrmate200ic5h_macro.xacro (robot description, xacro)
@@ -148,5 +148,5 @@
     <joint name="${prefix}link_5-tool0" type="fixed">
       <origin xyz="0 0 0" rpy="${pi} ${-pi/2.0} 0" />
-      <parent link="${prefix}link_5" />
+      <parent link="${prefix}flange" />
       <child link="${prefix}tool0" />
     </joint>

File: fanuc_lrmate200ic_support/urdf/lrmate200ic5hs_macro.xacro (robot description, xacro)
@@ -148,5 +148,5 @@
     <joint name="${prefix}link_5-tool0" type="fixed">
       <origin xyz="0 0 0" rpy="${pi} ${-pi/2.0} 0" />
-      <parent link="${prefix}link_5" />
+      <parent link="${prefix}flange" />
       <child link="${prefix}tool0" />
     </joint>

File: fanuc_lrmate200ic_support/urdf/lrmate200ic5l_macro.xacro (robot description, xacro)
@@ -170,5 +170,5 @@
     <joint name="${prefix}link_6-tool0" type="fixed">
       <origin xyz="0 0 0" rpy="${pi} ${-pi/2.0} 0" />
-      <parent link="${prefix}link_6" />
+      <parent link="${prefix}flange" />
       <child link="${prefix}tool0" />
     </joint>

File: fanuc_lrmate200ic_support/urdf/lrmate200ic_macro.xacro (robot description, xacro)
@@ -170,5 +170,5 @@
     <joint name="${prefix}link_6-tool0" type="fixed">
       <origin xyz="0 0 0" rpy="${pi} ${-pi/2.0} 0" />
-      <parent link="${prefix}link_6" />
+      <parent link="${prefix}flange" />
       <child link="${prefix}tool0" />
     </joint>

File: fanuc_m10ia_support/urdf/m10ia7l_macro.xacro (robot description, xacro)
@@ -170,5 +170,5 @@
     <joint name="${prefix}link_6-tool0" type="fixed">
       <origin xyz="0 0 0" rpy="${pi} ${-pi/2.0} 0" />
-      <parent link="${prefix}link_6" />
+      <parent link="${prefix}flange" />
       <child link="${prefix}tool0" />
     </joint>

File: fanuc_m10ia_support/urdf/m10ia_macro.xacro (robot description, xacro)
@@ -170,5 +170,5 @@
     <joint name="${prefix}link_6-tool0" type="fixed">
       <origin xyz="0 0 0" rpy="${pi} ${-pi/2.0} 0" />
-      <parent link="${prefix}link_6" />
+      <parent link="${prefix}flange" />
       <child link="${prefix}tool0" />
     </joint>

File: fanuc_m16ib_support/urdf/m16ib20_macro.xacro (robot description, xacro)
@@ -170,5 +170,5 @@
     <joint name="${prefix}link_6-tool0" type="fixed">
       <origin xyz="0 0 0" rpy="${pi} ${-pi/2.0} 0" />
-      <parent link="${prefix}link_6" />
+      <parent link="${prefix}flange" />
       <child link="${prefix}tool0" />
     </joint>

File: fanuc_m20ia_support/urdf/m20ia10l_macro.xacro (robot description, xacro)
@@ -170,5 +170,5 @@
     <joint name="${prefix}link_6-tool0" type="fixed">
       <origin xyz="0 0 0" rpy="${pi} ${-pi/2.0} 0" />
-      <parent link="${prefix}link_6" />
+      <parent link="${prefix}flange" />
       <child link="${prefix}tool0" />
     </joint>

File: fanuc_m20ia_support/urdf/m20ia_macro.xacro (robot description, xacro)
@@ -170,5 +170,5 @@
     <joint name="${prefix}link_6-tool0" type="fixed">
       <origin xyz="0 0 0" rpy="${pi} ${-pi/2.0} 0" />
-      <parent link="${prefix}link_6" />
+      <parent link="${prefix}flange" />
       <child link="${prefix}tool0" />
     </joint>

File: fanuc_m20ib_support/urdf/m20ib25_macro.xacro (robot description, xacro)
@@ -170,5 +170,5 @@
     <joint name="${prefix}link_6-tool0" type="fixed">
       <origin xyz="0 0 0" rpy="${pi} ${-pi/2.0} 0" />
-      <parent link="${prefix}link_6" />
+      <parent link="${prefix}flange" />
       <child link="${prefix}tool0" />
     </joint>

File: fanuc_m430ia_support/urdf/m430ia2f_macro.xacro (robot description, xacro)
@@ -146,4 +146,9 @@
     <!-- ROS-Industrial 'tool0' frame: all-zeros tool frame -->
     <link name="${prefix}tool0" />
+    <!-- Note: instead of 'flange', we use 'link_5' as parent of this frame
+               as it already has the correct orientation and location for
+               'tool0'. Using 'flange' here would require additional rotations
+               to undo the rotation introduced by 'joint_5-flange'.
+     -->
     <joint name="${prefix}link_5-tool0" type="fixed">
       <origin xyz="0 0 0" rpy="0 0 0" />

File: fanuc_m430ia_support/urdf/m430ia2p_macro.xacro (robot description, xacro)
@@ -168,4 +168,9 @@
     <!-- ROS-Industrial 'tool0' frame: all-zeros tool frame -->
     <link name="${prefix}tool0" />
+    <!-- Note: instead of 'flange', we use 'link_6' as parent of this frame
+               as it already has the correct orientation and location for
+               'tool0'. Using 'flange' here would require additional rotations
+               to undo the rotation introduced by 'joint_6-flange'.
+     -->
     <joint name="${prefix}link_6-tool0" type="fixed">
       <origin xyz="0 0 0" rpy="0 0 0" />

File: fanuc_m6ib_support/urdf/m6ib_macro.xacro (robot description, xacro)
@@ -170,5 +170,5 @@
     <joint name="${prefix}link_6-tool0" type="fixed">
       <origin xyz="0 0 0" rpy="${pi} ${-pi/2.0} 0" />
-      <parent link="${prefix}link_6" />
+      <parent link="${prefix}flange" />
       <child link="${prefix}tool0" />
     </joint>
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