Commit message: Reuse meshes of base model as much as possible.

File: fanuc_m6ib_support/urdf/m6ib6s_macro.xacro (robot description, xacro)
@@ -8,5 +8,5 @@
         <origin xyz="0 0 0" rpy="0 0 0"/>
         <geometry>
-          <mesh filename="package://fanuc_m6ib_support/meshes/m6ib6s/visual/base_link.stl"/>
+          <mesh filename="package://fanuc_m6ib_support/meshes/m6ib/visual/base_link.stl"/>
         </geometry>
         <xacro:material_fanuc_grey />
@@ -15,5 +15,5 @@
         <origin xyz="0 0 0" rpy="0 0 0"/>
         <geometry>
-          <mesh filename="package://fanuc_m6ib_support/meshes/m6ib6s/collision/base_link.stl"/>
+          <mesh filename="package://fanuc_m6ib_support/meshes/m6ib/collision/base_link.stl"/>
         </geometry>
       </collision>
@@ -23,5 +23,5 @@
         <origin xyz="0 0 0" rpy="0 0 0"/>
         <geometry>
-          <mesh filename="package://fanuc_m6ib_support/meshes/m6ib6s/visual/link_1.stl"/>
+          <mesh filename="package://fanuc_m6ib_support/meshes/m6ib/visual/link_1.stl"/>
         </geometry>
         <xacro:material_fanuc_yellow />
@@ -30,5 +30,5 @@
         <origin xyz="0 0 0" rpy="0 0 0"/>
         <geometry>
-          <mesh filename="package://fanuc_m6ib_support/meshes/m6ib6s/collision/link_1.stl"/>
+          <mesh filename="package://fanuc_m6ib_support/meshes/m6ib/collision/link_1.stl"/>
         </geometry>
       </collision>
@@ -53,5 +53,5 @@
         <origin xyz="0 0 0" rpy="0 0 0"/>
         <geometry>
-          <mesh filename="package://fanuc_m6ib_support/meshes/m6ib6s/visual/link_3.stl"/>
+          <mesh filename="package://fanuc_m6ib_support/meshes/m6ib/visual/link_3.stl"/>
         </geometry>
         <xacro:material_fanuc_yellow />
@@ -60,5 +60,5 @@
         <origin xyz="0 0 0" rpy="0 0 0"/>
         <geometry>
-          <mesh filename="package://fanuc_m6ib_support/meshes/m6ib6s/collision/link_3.stl"/>
+          <mesh filename="package://fanuc_m6ib_support/meshes/m6ib/collision/link_3.stl"/>
         </geometry>
       </collision>
@@ -83,5 +83,5 @@
         <origin xyz="0 0 0" rpy="0 0 0"/>
         <geometry>
-          <mesh filename="package://fanuc_m6ib_support/meshes/m6ib6s/visual/link_5.stl"/>
+          <mesh filename="package://fanuc_m6ib_support/meshes/m6ib/visual/link_5.stl"/>
         </geometry>
         <xacro:material_fanuc_yellow />
@@ -90,5 +90,5 @@
         <origin xyz="0 0 0" rpy="0 0 0"/>
         <geometry>
-          <mesh filename="package://fanuc_m6ib_support/meshes/m6ib6s/collision/link_5.stl"/>
+          <mesh filename="package://fanuc_m6ib_support/meshes/m6ib/collision/link_5.stl"/>
         </geometry>
       </collision>
@@ -98,5 +98,5 @@
         <origin xyz="0 0 0" rpy="0 0 0"/>
         <geometry>
-          <mesh filename="package://fanuc_m6ib_support/meshes/m6ib6s/visual/link_6.stl"/>
+          <mesh filename="package://fanuc_m6ib_support/meshes/m6ib/visual/link_6.stl"/>
         </geometry>
         <xacro:material_fanuc_black />
@@ -105,5 +105,5 @@
         <origin xyz="0 0 0" rpy="0 0 0"/>
         <geometry>
-          <mesh filename="package://fanuc_m6ib_support/meshes/m6ib6s/collision/link_6.stl"/>
+          <mesh filename="package://fanuc_m6ib_support/meshes/m6ib/collision/link_6.stl"/>
         </geometry>
       </collision>
