Commit message: Add experimental support for CR-7iA (ros-industrial/fanuc_experimental#35).

File: fanuc_cr7ia_support/urdf/cr7ia_macro.xacro (robot description, xacro)
@@ -2,5 +2,5 @@
 <robot xmlns:xacro="http://ros.org/wiki/xacro">
   <xacro:include filename="$(find fanuc_resources)/urdf/common_materials.xacro"/>
-  <xacro:macro name="fanuc_cr7ial" params="prefix">
+  <xacro:macro name="fanuc_cr7ia" params="prefix">
     <!-- links: main serial chain -->
     <link name="${prefix}base_link">
@@ -38,5 +38,5 @@
         <origin xyz="0 0 0" rpy="0 0 0"/>
         <geometry>
-          <mesh filename="package://fanuc_cr7ia_support/meshes/cr7ial/visual/link_2.stl"/>
+          <mesh filename="package://fanuc_cr7ia_support/meshes/cr7ia/visual/link_2.stl"/>
         </geometry>
         <xacro:material_fanuc_green />
@@ -45,5 +45,5 @@
         <origin xyz="0 0 0" rpy="0 0 0"/>
         <geometry>
-          <mesh filename="package://fanuc_cr7ia_support/meshes/cr7ial/collision/link_2.stl"/>
+          <mesh filename="package://fanuc_cr7ia_support/meshes/cr7ia/collision/link_2.stl"/>
         </geometry>
       </collision>
@@ -68,5 +68,5 @@
         <origin xyz="0 0 0" rpy="0 0 0"/>
         <geometry>
-          <mesh filename="package://fanuc_cr7ia_support/meshes/cr7ial/visual/link_4.stl"/>
+          <mesh filename="package://fanuc_cr7ia_support/meshes/cr7ia/visual/link_4.stl"/>
         </geometry>
         <xacro:material_fanuc_green />
@@ -75,5 +75,5 @@
         <origin xyz="0 0 0" rpy="0 0 0"/>
         <geometry>
-          <mesh filename="package://fanuc_cr7ia_support/meshes/cr7ial/collision/link_4.stl"/>
+          <mesh filename="package://fanuc_cr7ia_support/meshes/cr7ia/collision/link_4.stl"/>
         </geometry>
       </collision>
@@ -125,9 +125,9 @@
     </joint>
     <joint name="${prefix}joint_3" type="revolute">
-      <origin xyz="0 0 0.440" rpy="0 0 0" />
+      <origin xyz="0 0 0.330" rpy="0 0 0" />
       <parent link="${prefix}link_2" />
       <child link="${prefix}link_3" />
       <axis xyz="0 -1 0" />
-      <limit effort="0" lower="-0.802851" upper="3.10669" velocity="7.1558" />
+      <limit effort="0" lower="-0.7504911" upper="3.10669" velocity="7.1558" />
     </joint>
     <joint name="${prefix}joint_4" type="revolute">
@@ -139,5 +139,5 @@
     </joint>
     <joint name="${prefix}joint_5" type="revolute">
-      <origin xyz="0.420 0 0" rpy="0 0 0"/>
+      <origin xyz="0.335 0 0" rpy="0 0 0"/>
       <parent link="${prefix}link_4"/>
       <child link="${prefix}link_5"/>

Commit message: cr7ia: fix joint limits. Fix #310.
Based on the system variables, the limits for various joints were incorrect.

It could be Fanuc has changed the limits since the initial contribution of the support package.

File: fanuc_cr7ia_support/urdf/cr7ia_macro.xacro (robot description, xacro)
@@ -115,5 +115,5 @@
       <child link="${prefix}link_1" />
       <axis xyz="0 0 1" />
-      <limit effort="0" lower="-2.9671" upper="2.9671" velocity="6.4577" />
+      <limit effort="0" lower="-2.9671" upper="2.9671" velocity="7.8539" />
     </joint>
     <joint name="${prefix}joint_2" type="revolute">
@@ -122,5 +122,5 @@
       <child link="${prefix}link_2" />
       <axis xyz="0 1 0" />
-      <limit effort="0" lower="-1.15192" upper="1.74533" velocity="5.4105" />
+      <limit effort="0" lower="-1.1519" upper="1.7453" velocity="6.6322" />
     </joint>
     <joint name="${prefix}joint_3" type="revolute">
@@ -129,5 +129,5 @@
       <child link="${prefix}link_3" />
       <axis xyz="0 -1 0" />
-      <limit effort="0" lower="-0.7504911" upper="3.10669" velocity="7.1558" />
+      <limit effort="0" lower="-2.2621" upper="4.2586" velocity="9.0757" />
     </joint>
     <joint name="${prefix}joint_4" type="revolute">

File: fanuc_cr7ia_support/urdf/cr7ial_macro.xacro (robot description, xacro)
@@ -122,5 +122,5 @@
       <child link="${prefix}link_2" />
       <axis xyz="0 1 0" />
-      <limit effort="0" lower="-1.15192" upper="1.74533" velocity="5.4105" />
+      <limit effort="0" lower="-1.1519" upper="1.7453" velocity="5.4105" />
     </joint>
     <joint name="${prefix}joint_3" type="revolute">
@@ -129,5 +129,5 @@
       <child link="${prefix}link_3" />
       <axis xyz="0 -1 0" />
-      <limit effort="0" lower="-0.802851" upper="3.10669" velocity="7.1558" />
+      <limit effort="0" lower="-2.4397" upper="4.2586" velocity="7.1558" />
     </joint>
     <joint name="${prefix}joint_4" type="revolute">
